File: kello-yritys2.kicad_pcb (KiCad board)
At the start: 2 copper layers, 174 parts, among them J1 Conn_01x02_Male_To_Opto, J2 USB_B_Micro, J3 AVR-ISP-6, Q1 TEPT4400, Q10 BC850, Q11 BC850, Q12 BC850, Q13 BC850, Q14 BC850, Q15 BC850, Q16 BC850, Q17 BC850, Q18 BC850, Q19 BC850, Q2 IRLML6402, Q20 BC850, Q21 BC850, Q22 BC850, Q23 BC850, Q24 BC850, Q25 BC850, Q26 BC850, Q27 BC850, Q28 BC850, Q29 BC850, Q3 IRLML6402, Q30 BC850, Q31 BC850, Q32 BC850, Q33 BC850, Q4 IRLML6402, Q5 IRLML6402, Q6 BC850, Q7 BC850, Q8 BC850, Q9 BC850, SW1 SW_Push_Dual, SW2 SW_Push_Dual, U1 ATmega328PB-AU

Commit message: joo
Parts:
- D1, D10, D11, D12, D13, D14, D15, D16, D17, D18, D19, D2, D20, D21, D22, D23, D24, D25, D26, D27, D28, D29, D3, D30, D31, D32, D33, D34, D35, D36, D37, D38, D39, D4, D40, D41, D42, D43, D44, D45, D46, D47, D48, D49, D5, D50, D51, D52, D53, D54, D55, D56, D57, D58, D59, D6, D60, D61, D62, D63, D64, D65, D66, D67, D68, D69, D7, D70, D71, D72, D73, D74, D75, D76, D77, D78, D79, D8, D80, D81, D82, D9: footprint LED_THT:LED_D3.0mm_Clear -> LED_THT:LED_D3.0mm_Front
- J3: moved to B.Cu
- moved Q2 0.18 mm to (150.5, 24.8)
- moved Q3 0.13 mm to (108.6, 24.8)

Commit message: joo
Parts:
- moved R7 103.3 mm to (167.8, 111.6), turned to 270 degrees
- moved Q8 102.1 mm to (165.1, 106.0), turned to 90 degrees
- moved Q9 100.5 mm to (165.0, 102.5), turned to 180 degrees
- moved R8 99.2 mm to (165.1, 108.7)
- moved R39 71.1 mm to (184.5, 111.6), turned to 270 degrees
- moved R11 70.8 mm to (178.9, 111.6), turned to 270 degrees
- moved Q32 70.3 mm to (181.7, 106.2), turned to 90 degrees
- moved Q27 70.2 mm to (148.2, 102.5), turned to 180 degrees
- moved Q33 70.1 mm to (181.7, 102.6), turned to 180 degrees
- moved Q12 69.2 mm to (176.1, 106.2), turned to 90 degrees
- moved R40 68.1 mm to (181.7, 109.0)
- moved Q13 67.5 mm to (176.1, 102.6), turned to 180 degrees
- moved R27 66.9 mm to (151.0, 111.6), turned to 270 degrees
- moved R12 66.1 mm to (176.1, 109.0)
- moved R28 66.0 mm to (148.3, 108.8)
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Connections:
- J3 pad 1: /Naytto/Glo9 -> /Naytto/Glo1
- J3 pad 3: /Naytto/GloA -> /Naytto/Glo2
- J3 pad 4: /Naytto/Glo8 -> /Naytto/Glo0
- U1 pad 10: /Naytto/Glo3 -> /Naytto/Glo6
- U1 pad 11: /Naytto/Glo4 -> /Naytto/Glo7
- U1 pad 12: /Naytto/Glo5 -> /Naytto/GloA
- U1 pad 13: /Naytto/Glo6 -> /Naytto/Glo8
- U1 pad 14: /Naytto/Glo7 -> /Naytto/Glo9
- U1 pad 15: /Naytto/Glo8 -> /Naytto/Glo0
- U1 pad 16: /Naytto/Glo9 -> /Naytto/Glo1
- U1 pad 17: /Naytto/GloA -> /Naytto/Glo2
- U1 pad 7: /Naytto/Glo0 -> /Naytto/Glo4
- U1 pad 8: /Naytto/Glo1 -> /Naytto/Glo5
- U1 pad 9: /Naytto/Glo2 -> /Naytto/Glo3
Routing:
- net GNDREF: track 0.00 -> 148.8 mm
- net /Naytto/Numero/CatA: track 317.3 -> 358.0 mm
- net /Naytto/Numero/Cat8: track 303.4 -> 338.9 mm
- net /Naytto/Numero/Cat4: track 456.7 -> 487.0 mm
- net /Naytto/Numero/Cat9: track 340.5 -> 370.7 mm
- net /Naytto/sheet5E58E229/Collector: track 215.0 -> 185.6 mm
- net /Naytto/Numero/Cat5: track 308.4 -> 333.4 mm
- net /Naytto/Numero/Cat0: track 425.0 -> 450.0 mm
- net /Naytto/Numero/Cat3b: track 271.4 -> 291.3 mm
- net /Naytto/Numero/Cat1: track 476.4 -> 496.1 mm
- net /Naytto/Numero/Cat6a: track 202.7 -> 219.5 mm
- net /Naytto/Numero/Cat2: track 520.5 -> 534.9 mm
- net /Naytto/Numero/Cat6b: track 184.1 -> 197.9 mm
- net /Naytto/Numero/Cat7: track 217.8 -> 229.7 mm
- net Net-(Q10-Pad3): track 0.00 -> 9.46 mm
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
Commit message: joo
Parts:
- removed C2: 1n, Capacitor_SMD:C_0805_2012Metric
- removed R2: 150k, Resistor_SMD:R_0805_2012Metric
- added REF**: 0, Resistor_SMD:R_0805_2012Metric, F.Cu at (90.0, 23.9)
- added REF**: 0, Resistor_SMD:R_0805_2012Metric, F.Cu at (173.4, 114.3)
- added REF**: 0, Resistor_SMD:R_0805_2012Metric, F.Cu at (167.8, 114.3)
- added REF**: 0, Resistor_SMD:R_0805_2012Metric, F.Cu at (162.2, 114.3)
- added REF**: 0, Resistor_SMD:R_0805_2012Metric, F.Cu at (156.6, 114.3)
- added REF**: 0, Resistor_SMD:R_0805_2012Metric, F.Cu at (151.0, 114.3)
- added REF**: 0, Resistor_SMD:R_0805_2012Metric, F.Cu at (145.4, 114.3)
- added REF**: 0, Resistor_SMD:R_0805_2012Metric, F.Cu at (139.8, 114.3)
- added REF**: 0, Resistor_SMD:R_0805_2012Metric, F.Cu at (128.6, 114.3)
- moved C4 214.1 mm to (-1.02, 27.9), turned to 270 degrees
- moved C5 153.8 mm to (3.30, 23.6), turned to 270 degrees
- moved J3 104.2 mm to (87.6, 27.3), turned to 270 degrees
- moved C1 83.0 mm to (74.0, 116.3), turned to 270 degrees
- moved J2 82.1 mm to (56.5, 116.6), turned to 0 degrees
- moved Q32 78.2 mm to (103.4, 106.2)
- moved Q33 78.2 mm to (103.5, 102.6)
- moved R39 78.2 mm to (106.3, 111.6)
- moved R40 78.2 mm to (103.5, 109.0)
- moved U1 77.5 mm to (84.6, 113.0), turned to 90 degrees
- moved C7 70.9 mm to (36.6, 112.4)
- moved R92 70.9 mm to (36.6, 109.5)
- moved R93 70.9 mm to (36.6, 106.5)
- moved C6 66.9 mm to (63.7, 116.5)
- moved R90 66.9 mm to (63.7, 113.5)
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Connections:
- C1 pad 2: +5V -> Earth
- C3 pad 2: +5V -> Earth
- C4 pad 2: +5V -> Earth
- C5 pad 2: +5V -> Earth
- C6 pad 1: +5V -> Earth
- C7 pad 1: +5V -> Earth
- C8 pad 2: +5V -> Earth
- J1 pad 2: +5V -> Earth
- J2 pad 5: +5V -> Earth
- J2 pad 6: +5V -> Earth
- J3 pad 1: /Naytto/Glo1 -> /Naytto/Glo5
- J3 pad 3: /Naytto/Glo2 -> /Naytto/Glo4
- J3 pad 4: /Naytto/Glo0 -> /Naytto/Glo3
- J3 pad 6: +5V -> Earth
- Q1 pad 2: +5V -> Earth
- Q10 pad 2: GNDREF -> Earth
- Q12 pad 2: GNDREF -> Earth
- Q14 pad 2: GNDREF -> Earth
- Q16 pad 2: GNDREF -> Earth
- Q18 pad 2: GNDREF -> Earth
- Q20 pad 2: GNDREF -> Earth
- Q22 pad 2: GNDREF -> Earth
- Q24 pad 2: GNDREF -> Earth
- Q26 pad 2: GNDREF -> Earth
- Q28 pad 2: GNDREF -> Earth
- Q30 pad 2: GNDREF -> Earth
- Q32 pad 2: GNDREF -> Earth
- Q6 pad 2: GNDREF -> Earth
- Q8 pad 2: GNDREF -> Earth
- R10 pad 2: GNDREF -> Earth
- R12 pad 2: GNDREF -> Earth
- R14 pad 2: GNDREF -> Earth
- R16 pad 2: GNDREF -> Earth
- R20 pad 2: GNDREF -> Earth
- R22 pad 2: GNDREF -> Earth
- R24 pad 2: GNDREF -> Earth
- R26 pad 2: GNDREF -> Earth
- R28 pad 2: GNDREF -> Earth
- R30 pad 2: GNDREF -> Earth
- R38 pad 2: GNDREF -> Earth
- R40 pad 2: GNDREF -> Earth
- R6 pad 2: GNDREF -> Earth
- R8 pad 2: GNDREF -> Earth
- R90 pad 1: +5V -> Earth
- R92 pad 1: +5V -> Earth
- U1 pad 1: /Naytto/Ghi3 -> /Naytto/Ghi2
- U1 pad 10: /Naytto/Glo6 -> /Naytto/Glo9
- U1 pad 11: /Naytto/Glo7 -> /Naytto/Glo8
- U1 pad 13: /Naytto/Glo8 -> /Naytto/Glo7
- U1 pad 14: /Naytto/Glo9 -> /Naytto/Glo6
- U1 pad 15: /Naytto/Glo0 -> /Naytto/Glo3
- U1 pad 16: /Naytto/Glo1 -> /Naytto/Glo5
- U1 pad 17: /Naytto/Glo2 -> /Naytto/Glo4
- U1 pad 2: /Naytto/GloB -> /Naytto/Ghi3
- U1 pad 21: +5V -> Earth
- U1 pad 22: Net-(J2-Pad2) -> Net-(U1-Pad22)
- U1 pad 30: /Naytto/Ghi0 -> /Naytto/GloB
- U1 pad 31: /Naytto/Ghi1 -> /Naytto/Ghi0
- U1 pad 32: /Naytto/Ghi2 -> /Naytto/Ghi1
- U1 pad 5: +5V -> Earth
- U1 pad 7: /Naytto/Glo4 -> /Naytto/Glo2
- U1 pad 8: /Naytto/Glo5 -> /Naytto/Glo1
- U1 pad 9: /Naytto/Glo3 -> /Naytto/Glo0
Routing:
- net Earth: track 0.00 -> 327.2 mm, vias 0 -> 3
- net +5V: track 0.00 -> 243.9 mm
- net /Naytto/Ghi0: track 0.00 -> 172.5 mm, vias 0 -> 2
- net GNDREF: track 148.8 -> 0.00 mm
- net /Naytto/Ghi3: track 0.00 -> 148.2 mm
- net /Naytto/sheet5E58E229/Collector: track 185.6 -> 47.3 mm, vias 4 -> 0
- net /Naytto/Ghi1: track 0.00 -> 126.1 mm, vias 0 -> 2
- net /Naytto/Ghi2: track 0.00 -> 120.7 mm
- net /Naytto/Glo2: track 0.00 -> 94.4 mm
- net /Naytto/Glo1: track 0.00 -> 87.3 mm
- net /Naytto/Glo3: track 0.00 -> 81.3 mm
- net /Naytto/Glo0: track 0.00 -> 79.4 mm
- net /Naytto/Glo9: track 0.00 -> 73.7 mm
- net /Naytto/Glo8: track 0.00 -> 67.9 mm
- net /Naytto/GloA: track 0.00 -> 62.0 mm
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
Commit message: joo
Parts:
- moved C6 10.4 mm to (67.3, 106.7)
- moved J2 6.36 mm to (62.2, 119.4)
Routing:
- net /sheet5E8135E4/BtnOut: track 56.2 -> 31.0 mm
- net /DbdPb/BtnOut: track 25.6 -> 16.1 mm
- net Earth: track 327.2 -> 321.8 mm, vias 3 -> 9
Changed lines of the file:
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@@
     (thickness 1.6)
     (drawings 0)
-    (tracks 1357)
+    (tracks 1363)
     (zones 0)
     (modules 181)
@@
   )
   (setup
-    (last_trace_width 0.25)
+    (last_trace_width 2.5)
     (user_trace_width 0.35)
     (user_trace_width 0.5)
@@
   )
   (module Connector_USB:USB_Micro-B_Molex-105017-0001 (layer F.Cu)
-    (at 56.499 116.6185)
+    (at 62.23 119.38)
     (descr http://www.molex.com/pdm_docs/sd/1050170001_sd.pdf)
     (tags "Micro-USB SMD Typ-B")
@@
   )
   (module Capacitor_SMD:C_0805_2012Metric (layer F.Cu)
-    (at 63.7 116.457)
+    (at 67.31 106.68)
     (descr "Capacitor SMD 0805 (2012 Metric), square (rectangular) end terminal, IPC_7351 nominal, (Body size source: https://docs.google.com/spreadsheets/d/1BsfQQcO9C6DZCsRaXUlFlo91Tg2WpOkGARC1WS5S8t0/edit?usp=sharing), generated with kicad-footprint-generator")
     (tags capacitor)
@@
     )
   )
-  (segment (start 41.91 111.76) (end 82.55 111.76) (width 2.5) (layer B.Cu) (net 111))
+  (via (at 170.18 111.76) (size 2) (drill 1) (layers F.Cu B.Cu) (net 111))
+  (segment (start 41.91 111.76) (end 43.815 111.76) (width 2.5) (layer B.Cu) (net 111))
   (via (at 92.075 22.86) (size 0.8) (drill 0.4) (layers F.Cu B.Cu) (net 100))
   (via (at 94.361 22.86) (size 0.8) (drill 0.4) (layers F.Cu B.Cu) (net 100))
@@
   (segment (start 74.041 115.382) (end 74.041 113.632) (width 0.5) (layer F.Cu) (net 1))
   (segment (start 83.6445 119.38) (end 83.077482 119.947018) (width 0.5) (layer F.Cu) (net 1))
-  (segment (start 74.11599 110.557) (end 64.6375 110.557) (width 0.25) (layer F.Cu) (net 2))
-  (segment (start 83.382 118.13815) (end 82.148142 119.372008) (width 0.25) (layer F.Cu) (net 2))
-  (segment (start 79.797784 119.372008) (end 75.31899 114.893214) (width 0.25) (layer F.Cu) (net 2))
-  (segment (start 83.382 117.28) (end 83.382 118.13815) (width 0.25) (layer F.Cu) (net 2))
   (segment (start 75.31899 111.76) (end 74.11599 110.557) (width 0.25) (layer F.Cu) (net 2))
   (segment (start 82.148142 119.372008) (end 79.797784 119.372008) (width 0.25) (layer F.Cu) (net 2))
+  (segment (start 79.797784 119.372008) (end 75.31899 114.893214) (width 0.25) (layer F.Cu) (net 2))
+  (segment (start 83.382 118.13815) (end 82.148142 119.372008) (width 0.25) (layer F.Cu) (net 2))
   (segment (start 75.31899 114.893214) (end 75.31899 111.76) (width 0.25) (layer F.Cu) (net 2))
+  (segment (start 83.382 117.28) (end 83.382 118.13815) (width 0.25) (layer F.Cu) (net 2))
   (segment (start 64.897 114.935) (end 61.722 114.935) (width 0.25) (layer F.Cu) (net 3))
   (segment (start 85.782 118.13815) (end 86.487 118.84315) (width 0.25) (layer F.Cu) (net 3))
   (segment (start 85.782 117.28) (end 85.782 118.13815) (width 0.25) (layer F.Cu) (net 3))
-  (segment (start 61.722 114.935) (end 59.2 112.413) (width 0.25) (layer F.Cu) (net 3))
   (segment (start 86.487 119.91685) (end 84.99185 121.412) (width 0.25) (layer F.Cu) (net 3))
   (segment (start 86.487 118.84315) (end 86.487 119.91685) (width 0.25) (layer F.Cu) (net 3))
   (segment (start 84.99185 121.412) (end 71.374 121.412) (width 0.25) (layer F.Cu) (net 3))
   (segment (start 71.374 121.412) (end 64.897 114.935) (width 0.25) (layer F.Cu) (net 3))
-  (segment (start 37.5845 112.413) (end 59.2 112.413) (width 0.25) (layer F.Cu) (net 3))
   (via (at 172.974 86.106) (size 0.8) (drill 0.4) (layers F.Cu B.Cu) (net 20))
   (via (at 173.736 87.122) (size 0.8) (drill 0.4) (layers F.Cu B.Cu) (net 21))
@@
   (segment (start 160.3225 107.0575) (end 160.335 107.045) (width 0.5) (layer F.Cu) (net 111))
   (segment (start 160.3225 108.839) (end 160.3225 107.0575) (width 0.5) (layer F.Cu) (net 111))
-  (segment (start 171.4985 108.839) (end 171.4985 110.7925) (width 0.5) (layer F.Cu) (net 111))
-  (segment (start 177.0865 110.520126) (end 177.0865 108.966) (width 0.5) (layer F.Cu) (net 111))
-  (segment (start 178.199374 111.633) (end 177.0865 110.520126) (width 0.5) (layer F.Cu) (net 111))
-  (segment (start 172.339 111.633) (end 171.4985 110.7925) (width 0.5) (layer F.Cu) (net 111))
-  (segment (start 178.199374 111.633) (end 172.339 111.633) (width 0.5) (layer F.Cu) (net 111))
   (segment (start 166.0375 109.412) (end 166.0375 108.712) (width 0.5) (layer F.Cu) (net 111))
   (segment (start 167.023374 111.633) (end 166.0375 110.647126) (width 0.5) (layer F.Cu) (net 111))
   (segment (start 166.0375 110.647126) (end 166.0375 109.412) (width 0.5) (layer F.Cu) (net 111))
-  (segment (start 172.339 111.633) (end 167.023374 111.633) (width 0.5) (layer F.Cu) (net 111))
   (segment (start 160.3225 109.539) (end 160.3225 108.839) (width 0.5) (layer F.Cu) (net 111))
   (segment (start 160.3225 110.520126) (end 160.3225 109.539) (width 0.5) (layer F.Cu) (net 111))
@@
   (segment (start 102.108 111.633) (end 100.838 111.633) (width 0.5) (layer F.Cu) (net 111))
   (segment (start 105.537 111.633) (end 102.108 111.633) (width 0.5) (layer F.Cu) (net 111))
-  (segment (start 180.594 111.633) (end 180.721 111.633) (width 0.5) (layer F.Cu) (net 111))
-  (segment (start 180.594 111.633) (end 178.199374 111.633) (width 0.5) (layer F.Cu) (net 111))
-  (via (at 181.61 111.76) (size 2) (drill 1) (layers F.Cu B.Cu) (net 111))
-  (segment (start 100.33 111.76) (end 182.88 111.76) (width 2.5) (layer B.Cu) (net 111))
+  (segment (start 100.33 111.76) (end 170.2 111.76) (width 2.5) (layer B.Cu) (net 111))
   (via (at 100.33 111.76) (size 2) (drill 1) (layers F.Cu B.Cu) (net 111))
   (segment (start 100.711 111.76) (end 100.838 111.633) (width 0.5) (layer F.Cu) (net 111))
   (segment (start 100.33 111.76) (end 100.711 111.76) (width 0.5) (layer F.Cu) (net 111))
-  (segment (start 180.848 111.76) (end 180.721 111.633) (width 0.5) (layer F.Cu) (net 111))
-  (segment (start 181.61 111.76) (end 180.848 111.76) (width 0.5) (layer F.Cu) (net 111))
   (segment (start 82.55 111.76) (end 100.33 111.76) (width 2.5) (layer B.Cu) (net 111))
   (via (at 82.55 111.76) (size 2) (drill 1) (layers F.Cu B.Cu) (net 111))
@@
   (segment (start 84.182 110.128) (end 84.182 108.78) (width 0.5) (layer F.Cu) (net 111))
   (segment (start 82.55 111.76) (end 84.182 110.128) (width 0.5) (layer F.Cu) (net 111))
+  (segment (start 171.4985 110.4415) (end 170.18 111.76) (width 0.5) (layer F.Cu) (net 111))
+  (segment (start 171.4985 108.839) (end 171.4985 110.4415) (width 0.5) (layer F.Cu) (net 111))
+  (segment (start 177.0865 110.4415) (end 177.0865 108.966) (width 0.5) (layer F.Cu) (net 111))
+  (segment (start 167.023374 111.633) (end 175.895 111.633) (width 0.5) (layer F.Cu) (net 111))
+  (segment (start 175.895 111.633) (end 177.0865 110.4415) (width 0.5) (layer F.Cu) (net 111))
+  (segment (start 41.91 111.76) (end 31.75 111.76) (width 2.5) (layer B.Cu) (net 111))
+  (segment (start 31.75 111.76) (end 29.21 111.76) (width 2.5) (layer B.Cu) (net 111))
+  (segment (start 69.215 111.76) (end 82.55 111.76) (width 2.5) (layer B.Cu) (net 111))
+  (via (at 69.215 111.76) (size 2) (drill 1) (layers F.Cu B.Cu) (net 111))
+  (segment (start 60.325 111.76) (end 69.215 111.76) (width 2.5) (layer B.Cu) (net 111))
+  (via (at 60.325 111.76) (size 2) (drill 1) (layers F.Cu B.Cu) (net 111))
+  (segment (start 53.975 111.76) (end 60.325 111.76) (width 2.5) (layer B.Cu) (net 111))
+  (via (at 53.975 111.76) (size 2) (drill 1) (layers F.Cu B.Cu) (net 111))
+  (segment (start 49.53 111.76) (end 53.975 111.76) (width 2.5) (layer B.Cu) (net 111))
+  (via (at 49.53 111.76) (size 2) (drill 1) (layers F.Cu B.Cu) (net 111))
+  (segment (start 46.355 111.76) (end 49.53 111.76) (width 2.5) (layer B.Cu) (net 111))
+  (via (at 46.355 111.76) (size 2) (drill 1) (layers F.Cu B.Cu) (net 111))
+  (segment (start 43.815 111.76) (end 46.355 111.76) (width 2.5) (layer B.Cu) (net 111))
+  (via (at 43.815 111.76) (size 2) (drill 1) (layers F.Cu B.Cu) (net 111))
   (segment (start 88.454 104.9805) (end 89.154 104.9805) (width 0.25) (layer F.Cu) (net 112))
   (segment (start 87.49265 104.9805) (end 88.454 104.9805) (width 0.25) (layer F.Cu) (net 112))

Commit message: joo
Parts:
- removed the REF** at (90.0, 23.9)
- added REF**: 0, Resistor_SMD:R_0805_2012Metric, F.Cu at (91.1, 109.9)
- added REF**: 0, Resistor_SMD:R_0805_2012Metric, F.Cu at (88.4, 98.8)
- added REF**: 0, Resistor_SMD:R_0805_2012Metric, F.Cu at (93.7, 109.9)
- added REF**: 0, Resistor_SMD:R_0805_2012Metric, F.Cu at (86.9, 35.3)
- added REF**: 0, Resistor_SMD:R_0805_2012Metric, F.Cu at (95.5, 107.8)
- added REF**: 0, Resistor_SMD:R_0805_2012Metric, F.Cu at (95.5, 105.9)
- added REF**: 0, Resistor_SMD:R_0805_2012Metric, F.Cu at (63.8, 114.0)
- moved R93 26.8 mm to (63.0, 111.3)
- moved C7 25.8 mm to (61.7, 106.4), turned to 90 degrees
- moved SW1 25.5 mm to (66.0, 109.2), turned to 90 degrees
- moved R92 22.7 mm to (59.2, 106.4), turned to 90 degrees
- moved R31 14.8 mm to (99.6, 24.6), turned to 180 degrees
- moved R32 13.5 mm to (98.8, 27.4), turned to 90 degrees
- moved R91 10.5 mm to (74.2, 109.7), turned to 90 degrees
- moved R90 9.80 mm to (67.3, 104.4), turned to 270 degrees
- moved SW2 8.58 mm to (57.9, 109.2), turned to 90 degrees
- moved Q3 7.48 mm to (101.6, 27.4), turned to 0 degrees
- moved C6 3.42 mm to (69.8, 104.4), turned to 270 degrees
- moved J2 1.27 mm to (62.2, 120.7)
- moved C4 1.02 mm to (0.00, 27.9), turned to 90 degrees
- moved C5 0.57 mm to (2.79, 23.4), turned to 180 degrees
- moved R4 0.56 mm to (85.7, 102.9)
Connections:
- U1 pad 31: /Naytto/Ghi0 -> /Naytto/Ghi1
- U1 pad 32: /Naytto/Ghi1 -> /Naytto/Ghi0
Routing:
- net Earth: track 321.8 -> 1005.7 mm
- net +5V: track 243.9 -> 405.9 mm
- net /Naytto/Glo3: track 81.3 -> 187.3 mm, vias 0 -> 2
- net /Naytto/Glo4: track 28.0 -> 121.1 mm
- net Net-(J3-Pad5): track 13.9 -> 105.0 mm
- net /Naytto/Glo5: track 32.0 -> 122.8 mm
- net (no net): track 0.00 -> 18.4 mm
- net /DbdPb/BtnOut: track 16.1 -> 31.3 mm
- net /Naytto/Ghi1: track 126.1 -> 111.5 mm
- net /sheet5E8135E4/BtnOut: track 31.0 -> 42.9 mm
- net Net-(R90-Pad2): track 0.00 -> 10.5 mm
- net Net-(R92-Pad2): track 0.00 -> 9.60 mm
- net /Naytto/GloB: track 52.3 -> 54.3 mm
- net /Naytto/Ghi0: track 172.5 -> 174.3 mm
- net /Naytto/Numero/Cat3a: track 695.4 -> 696.9 mm
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
Commit message: joo
Parts:
- removed the REF** at (91.1, 109.9)
- removed the REF** at (162.2, 114.3)
- removed the REF** at (156.6, 114.3)
- removed the REF** at (151.0, 114.3)
- removed the REF** at (145.4, 114.3)
- removed the REF** at (139.8, 114.3)
- removed the REF** at (128.6, 114.3)
- removed the REF** at (88.4, 98.8)
- removed the REF** at (93.7, 109.9)
- removed the REF** at (95.5, 107.8)
- removed the REF** at (173.4, 114.3)
- removed the REF** at (167.8, 114.3)
- added R2: 1M, Resistor_SMD:R_0805_2012Metric, F.Cu at (51.7, 109.7)
- added REF**: 0, Resistor_SMD:R_0805_2012Metric, F.Cu at (90.4, 100.1)
- added REF**: 0, Resistor_SMD:R_0805_2012Metric, F.Cu at (91.1, 110.2)
- added REF**: 0, Resistor_SMD:R_0805_2012Metric, F.Cu at (87.0, 98.9)
- added REF**: 0, Resistor_SMD:R_0805_2012Metric, F.Cu at (93.9, 110.4)
- added REF**: 0, Resistor_SMD:R_0805_2012Metric, F.Cu at (95.5, 108.1)
- Q1: footprint LED_THT:LED_D3.0mm_Clear -> LED_THT:LED_D3.0mm_Front
- moved R4 3.10 mm to (83.2, 104.6), turned to 0 degrees
- moved Q1 2.62 mm to (90.2, 102.9), turned to 180 degrees
- moved J1 2.22 mm to (93.5, 100.1)
- moved R3 0.28 mm to (91.2, 105.9)
Routing:
- net (no net): track 18.4 -> 0.00 mm
- net +5V: track 405.9 -> 413.5 mm
- net /Naytto/GloB: track 54.3 -> 60.8 mm
- net Net-(Q1-Pad1): track 24.9 -> 19.1 mm
- net Earth: track 1005.7 -> 1010.9 mm
- net /Naytto/Glo3: track 187.3 -> 192.5 mm, vias 2 -> 4
- net /Naytto/Glo2: track 94.4 -> 91.2 mm
- net Net-(J3-Pad5): track 105.0 -> 102.0 mm
- net /Naytto/Glo1: track 87.3 -> 84.4 mm
- net Net-(J1-Pad1): track 12.4 -> 14.5 mm
- net /Naytto/Glo4: track 121.1 -> 122.5 mm

Commit message: joo
Routing:
- net +5V: track 413.5 -> 417.9 mm
Changed lines of the file:
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@@
   )
   (setup
-    (last_trace_width 1.5)
+    (last_trace_width 0.5)
     (user_trace_width 0.35)
     (user_trace_width 0.5)
@@
   (segment (start 96.770959 102.176809) (end 96.058973 102.888795) (width 0.25) (layer F.Cu) (net 1))
   (segment (start 96.058973 102.888795) (end 96.058972 103.964618) (width 0.25) (layer F.Cu) (net 1))
-  (segment (start 3.7315 23.368) (end 4.1285 23.765) (width 0.75) (layer F.Cu) (net 1))
   (segment (start 2.00401 25.93599) (end 3.7315 24.2085) (width 1.5) (layer F.Cu) (net 1))
   (segment (start 0.254 30.64) (end 2.00401 28.88999) (width 1.5) (layer F.Cu) (net 1))
@@
   (segment (start 91.981998 22.606) (end 90.711998 21.336) (width 1.5) (layer F.Cu) (net 1))
   (segment (start 90.711998 21.336) (end 6.604 21.336) (width 1.5) (layer F.Cu) (net 1))
+  (segment (start 4.1285 23.765) (end 3.7315 23.368) (width 1) (layer F.Cu) (net 1))
+  (segment (start 8.575 23.765) (end 4.1285 23.765) (width 1) (layer F.Cu) (net 1))
   (segment (start 75.31899 114.893214) (end 75.31899 109.94149) (width 0.25) (layer F.Cu) (net 2))
   (segment (start 75.31899 109.94149) (end 74.168 108.7905) (width 0.25) (layer F.Cu) (net 2))
@@
   (segment (start 103.449 104.622) (end 104.505 103.566) (width 0.5) (layer F.Cu) (net 89))
   (segment (start 103.449 105.182) (end 103.449 104.622) (width 0.5) (layer F.Cu) (net 89))
-  (segment (start 106.299 110.335) (end 106.299 110.8225) (width 0.5) (layer F.Cu) (net 89))
-  (segment (start 104.349 105.182) (end 106.299 107.132) (width 0.5) (layer F.Cu) (net 89))
-  (segment (start 103.449 105.182) (end 104.349 105.182) (width 0.5) (layer F.Cu) (net 89))
-  (segment (start 106.299 107.132) (end 106.299 110.335) (width 0.5) (layer F.Cu) (net 89))
+  (segment (start 104.349 105.182) (end 103.449 105.182) (width 0.5) (layer F.Cu) (net 89))
+  (segment (start 106.299 110.6955) (end 106.299 107.132) (width 0.5) (layer F.Cu) (net 89))
+  (segment (start 106.299 107.132) (end 104.349 105.182) (width 0.5) (layer F.Cu) (net 89))
   (segment (start 102.499 104.471998) (end 102.499 106.232) (width 0.5) (layer F.Cu) (net 90))
   (segment (start 103.505 103.465998) (end 102.499 104.471998) (width 0.5) (layer F.Cu) (net 90))

Commit message: joo
Parts:
- moved R2 7.30 mm to (53.3, 116.8)
- moved R93 5.08 mm to (67.1, 114.3), turned to 270 degrees
- moved C7 4.45 mm to (57.3, 106.4)
- moved R92 4.45 mm to (54.7, 106.4)
- moved SW2 4.45 mm to (53.5, 109.2)
- moved SW1 3.81 mm to (62.2, 109.2)
- moved R90 3.81 mm to (63.5, 104.4)
- moved C6 3.81 mm to (66.0, 104.4)
Routing:
- net Earth: track 1010.9 -> 1002.6 mm
- net /DbdPb/BtnOut: track 31.3 -> 36.7 mm
- net +5V: track 417.9 -> 421.9 mm
- net /sheet5E8135E4/BtnOut: track 42.9 -> 45.4 mm
