File: kello-yritys2.kicad_pcb (KiCad board)
At the start: 2 copper layers, 181 parts, among them J1 Conn_01x02_Male_To_Opto, J2 USB_B_Micro, J3 AVR-ISP-6, Q1 TEPT4400, Q10 BC850, Q11 BC850, Q12 BC850, Q13 BC850, Q14 BC850, Q15 BC850, Q16 BC850, Q17 BC850, Q18 BC850, Q19 BC850, Q2 IRLML6402, Q20 BC850, Q21 BC850, Q22 BC850, Q23 BC850, Q24 BC850, Q25 BC850, Q26 BC850, Q27 BC850, Q28 BC850, Q29 BC850, Q3 IRLML6402, Q30 BC850, Q31 BC850, Q32 BC850, Q33 BC850, Q4 IRLML6402, Q5 IRLML6402, Q6 BC850, Q7 BC850, Q8 BC850, Q9 BC850, SW1 SW_Push_Dual, SW2 SW_Push_Dual, U1 ATmega328PB-AU

Commit message: joo
Parts:
- removed R2: 1M, Resistor_SMD:R_0805_2012Metric
- added R41: 1M, Resistor_SMD:R_0805_2012Metric, F.Cu at (36.6, 100.8)
- added R42: 1M, Resistor_SMD:R_0805_2012Metric, F.Cu at (38.6, 100.8)
- added R43: 1M, Resistor_SMD:R_0805_2012Metric, F.Cu at (40.6, 100.8)
- added R44: 1M, Resistor_SMD:R_0805_2012Metric, F.Cu at (42.7, 100.8)
- added R45: 1M, Resistor_SMD:R_0805_2012Metric, F.Cu at (21.6, 98.0)
- added R46: 1M, Resistor_SMD:R_0805_2012Metric, F.Cu at (21.6, 94.0)
- added R47: 1M, Resistor_SMD:R_0805_2012Metric, F.Cu at (21.6, 96.0)
- added R48: 1M, Resistor_SMD:R_0805_2012Metric, F.Cu at (24.4, 100.8)
- added R49: 1M, Resistor_SMD:R_0805_2012Metric, F.Cu at (26.4, 100.8)
- added R50: 1M, Resistor_SMD:R_0805_2012Metric, F.Cu at (28.4, 100.8)
- added R51: 1M, Resistor_SMD:R_0805_2012Metric, F.Cu at (32.5, 100.8)
- added R52: 1M, Resistor_SMD:R_0805_2012Metric, F.Cu at (34.5, 100.8)
- added R53: 1M, Resistor_SMD:R_0805_2012Metric, F.Cu at (30.5, 100.8)
Routing:
- net Earth: track 1002.6 -> 1043.2 mm, vias 9 -> 6
- net /Naytto/Numero/Cat3b: track 291.3 -> 306.4 mm
- net /Naytto/Numero/Cat6a: track 219.5 -> 234.4 mm
- net /Naytto/Numero/Cat5: track 333.4 -> 347.4 mm
- net /Naytto/Numero/Cat6b: track 197.9 -> 211.3 mm
- net /Naytto/Numero/Cat4: track 487.0 -> 499.7 mm
- net /Naytto/Numero/Cat7: track 229.7 -> 241.4 mm
- net /Naytto/Numero/CatA: track 358.0 -> 368.3 mm
- net /Naytto/Numero/Cat8: track 338.9 -> 347.6 mm
- net /Naytto/Numero/Cat9: track 370.7 -> 377.8 mm
- net /Naytto/Numero/Cat0: track 450.1 -> 455.7 mm
- net /Naytto/Numero/Cat1: track 496.1 -> 500.2 mm
- net /Naytto/Numero/Cat2: track 534.9 -> 538.1 mm
- net +5V: track 421.9 -> 418.9 mm
- net /Naytto/Numero/Cat3a: track 696.9 -> 699.1 mm

Commit message: joo
Parts:
- moved R11 1.89 mm to (177.2, 111.0), turned to 180 degrees
- moved REF** 1.78 mm to (85.1, 35.3), turned to 180 degrees
- moved J3 1.27 mm to (86.4, 27.3)
Routing:
- net Earth: track 1043.2 -> 973.7 mm, vias 6 -> 17
- net /Naytto/Glo3: track 192.5 -> 200.4 mm, vias 4 -> 2
- net /Naytto/Glo6: track 50.5 -> 53.4 mm
- net /Naytto/Ghi1: track 111.5 -> 113.1 mm
- net /Naytto/Glo4: track 122.5 -> 121.0 mm
- net +5V: track 418.9 -> 420.4 mm
- net /Naytto/Ghi0: track 174.3 -> 175.7 mm
- net Net-(J3-Pad5): track 102.0 -> 101.1 mm
- net /Naytto/Glo5: track 123.1 -> 123.9 mm

Commit message: joo
Parts:
- removed the REF** at (90.4, 100.1)
- removed the REF** at (91.1, 110.2)
- removed the REF** at (87.0, 98.9)
- removed the REF** at (93.9, 110.4)
- removed the REF** at (85.1, 35.3)
- removed the REF** at (95.5, 108.1)
- added REF**: 0, Resistor_SMD:R_0805_2012Metric, F.Cu at (107.6, 93.7)
- added REF**: 0, Resistor_SMD:R_0805_2012Metric, F.Cu at (108.2, 103.9)
- added REF**: 0, Resistor_SMD:R_0805_2012Metric, F.Cu at (104.1, 92.6)
- added REF**: 0, Resistor_SMD:R_0805_2012Metric, F.Cu at (111.0, 104.0)
- added REF**: 0, Resistor_SMD:R_0805_2012Metric, F.Cu at (102.2, 29.0)
- added REF**: 0, Resistor_SMD:R_0805_2012Metric, F.Cu at (112.6, 101.7)
-  : renamed from J3
- moved Q21 18.3 mm to (143.0, 96.1)
- moved Q22 18.3 mm to (148.6, 99.7)
- moved Q23 18.3 mm to (148.6, 96.1)
- moved Q24 18.3 mm to (154.2, 99.7)
- moved Q25 18.3 mm to (154.2, 96.1)
- moved Q27 18.3 mm to (165.4, 96.1)
- moved Q29 18.3 mm to (170.9, 96.1)
- moved Q6 18.3 mm to (176.5, 99.7)
- moved Q7 18.3 mm to (176.5, 96.1)
- moved R1 18.3 mm to (106.3, 99.6)
- moved R11 18.3 mm to (194.3, 104.6)
- moved R8 18.3 mm to (182.2, 102.4)
- moved C1 18.3 mm to (91.2, 110.0)
- moved C3 18.3 mm to (101.7, 113.0)
- moved D10 18.3 mm to (188.6, 21.3)
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Other:
- board outline added: 189.2 x 105.4 mm

Commit message: joo
Parts:
- added C2: 100nF, Capacitor_SMD:C_0805_2012Metric, F.Cu at (70.6, 110.7)
- added C9: 100uF, Capacitor_SMD:CP_Elec_6.3x7.7, F.Cu at (66.0, 108.0)
- J3: renamed from  
Routing:
- net Earth: track 973.7 -> 976.3 mm
- net +5V: track 420.4 -> 422.4 mm
Changed lines of the file:
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@@
     (thickness 1.6)
     (drawings 4)
-    (tracks 1648)
+    (tracks 1653)
     (zones 0)
-    (modules 193)
+    (modules 195)
     (nets 114)
   )
@@
   )
   (setup
-    (last_trace_width 0.25)
+    (last_trace_width 0.5)
     (user_trace_width 0.35)
     (user_trace_width 0.5)
@@
     (add_net "Net-(U1-Pad28)")
   )
+  (module Capacitor_SMD:CP_Elec_6.3x7.7 (layer F.Cu)
+    (at 66.04 107.95 180)
+    (descr "SMD capacitor, aluminum electrolytic, Nichicon, 6.3x7.7mm")
+    (tags "capacitor electrolytic")
+    (attr smd)
+    (fp_text reference C9 (at 0 -4.35) (layer F.SilkS)
+      (effects (font (size 1 1) (thickness 0.15)))
+    )
+    (fp_text value 100uF (at 0 4.35) (layer F.Fab)
+      (effects (font (size 1 1) (thickness 0.15)))
+    )
+    (fp_text user %R (at 0 0) (layer F.Fab)
+      (effects (font (size 1 1) (thickness 0.15)))
+    )
+    (fp_line (start -4.7 1.05) (end -3.55 1.05) (layer F.CrtYd) (width 0.05))
+    (fp_line (start -4.7 -1.05) (end -4.7 1.05) (layer F.CrtYd) (width 0.05))
+    (fp_line (start -3.55 -1.05) (end -4.7 -1.05) (layer F.CrtYd) (width 0.05))
+    (fp_line (start -3.55 1.05) (end -3.55 2.4) (layer F.CrtYd) (width 0.05))
+    (fp_line (start -3.55 -2.4) (end -3.55 -1.05) (layer F.CrtYd) (width 0.05))
+    (fp_line (start -3.55 -2.4) (end -2.4 -3.55) (layer F.CrtYd) (width 0.05))
+    (fp_line (start -3.55 2.4) (end -2.4 3.55) (layer F.CrtYd) (width 0.05))
+    (fp_line (start -2.4 -3.55) (end 3.55 -3.55) (layer F.CrtYd) (width 0.05))
+    (fp_line (start -2.4 3.55) (end 3.55 3.55) (layer F.CrtYd) (width 0.05))
+    (fp_line (start 3.55 1.05) (end 3.55 3.55) (layer F.CrtYd) (width 0.05))
+    (fp_line (start 4.7 1.05) (end 3.55 1.05) (layer F.CrtYd) (width 0.05))
+    (fp_line (start 4.7 -1.05) (end 4.7 1.05) (layer F.CrtYd) (width 0.05))
+    (fp_line (start 3.55 -1.05) (end 4.7 -1.05) (layer F.CrtYd) (width 0.05))
+    (fp_line (start 3.55 -3.55) (end 3.55 -1.05) (layer F.CrtYd) (width 0.05))
+    (fp_line (start -4.04375 -2.24125) (end -4.04375 -1.45375) (layer F.SilkS) (width 0.12))
+    (fp_line (start -4.4375 -1.8475) (end -3.65 -1.8475) (layer F.SilkS) (width 0.12))
+    (fp_line (start -3.41 2.345563) (end -2.345563 3.41) (layer F.SilkS) (width 0.12))
+    (fp_line (start -3.41 -2.345563) (end -2.345563 -3.41) (layer F.SilkS) (width 0.12))
+    (fp_line (start -3.41 -2.345563) (end -3.41 -1.06) (layer F.SilkS) (width 0.12))
+    (fp_line (start -3.41 2.345563) (end -3.41 1.06) (layer F.SilkS) (width 0.12))
+    (fp_line (start -2.345563 3.41) (end 3.41 3.41) (layer F.SilkS) (width 0.12))
+    (fp_line (start -2.345563 -3.41) (end 3.41 -3.41) (layer F.SilkS) (width 0.12))
+    (fp_line (start 3.41 -3.41) (end 3.41 -1.06) (layer F.SilkS) (width 0.12))
+    (fp_line (start 3.41 3.41) (end 3.41 1.06) (layer F.SilkS) (width 0.12))
+    (fp_line (start -2.389838 -1.645) (end -2.389838 -1.015) (layer F.Fab) (width 0.1))
+    (fp_line (start -2.704838 -1.33) (end -2.074838 -1.33) (layer F.Fab) (width 0.1))
+    (fp_line (start -3.3 2.3) (end -2.3 3.3) (layer F.Fab) (width 0.1))
+    (fp_line (start -3.3 -2.3) (end -2.3 -3.3) (layer F.Fab) (width 0.1))
+    (fp_line (start -3.3 -2.3) (end -3.3 2.3) (layer F.Fab) (width 0.1))
+    (fp_line (start -2.3 3.3) (end 3.3 3.3) (layer F.Fab) (width 0.1))
+    (fp_line (start -2.3 -3.3) (end 3.3 -3.3) (layer F.Fab) (width 0.1))
+    (fp_line (start 3.3 -3.3) (end 3.3 3.3) (layer F.Fab) (width 0.1))
+    (fp_circle (center 0 0) (end 3.15 0) (layer F.Fab) (width 0.1))
+    (pad 2 smd roundrect (at 2.7 0 180) (size 3.5 1.6) (layers F.Cu F.Paste F.Mask) (roundrect_rratio 0.15625)
+      (net 111 Earth))
+    (pad 1 smd roundrect (at -2.7 0 180) (size 3.5 1.6) (layers F.Cu F.Paste F.Mask) (roundrect_rratio 0.15625)
+      (net 1 +5V))
+    (model ${KISYS3DMOD}/Capacitor_SMD.3dshapes/CP_Elec_6.3x7.7.wrl
+      (at (xyz 0 0 0))
+      (scale (xyz 1 1 1))
+      (rotate (xyz 0 0 0))
+    )
+  )
+  (module Capacitor_SMD:C_0805_2012Metric (layer F.Cu)
+    (at 70.612 110.744 270)
+    (descr "Capacitor SMD 0805 (2012 Metric), square (rectangular) end terminal, IPC_7351 nominal, (Body size source: https://docs.google.com/spreadsheets/d/1BsfQQcO9C6DZCsRaXUlFlo91Tg2WpOkGARC1WS5S8t0/edit?usp=sharing), generated with kicad-footprint-generator")
+    (tags capacitor)
+    (attr smd)
+    (fp_text reference C2 (at 0 -1.65 90) (layer F.SilkS)
+      (effects (font (size 1 1) (thickness 0.15)))
+    )
+    (fp_text value 100nF (at 0 1.65 90) (layer F.Fab)
+      (effects (font (size 1 1) (thickness 0.15)))
+    )
+    (fp_text user %R (at 0 0 90) (layer F.Fab)
+      (effects (font (size 0.5 0.5) (thickness 0.08)))
+    )
+    (fp_line (start 1.68 0.95) (end -1.68 0.95) (layer F.CrtYd) (width 0.05))
+    (fp_line (start 1.68 -0.95) (end 1.68 0.95) (layer F.CrtYd) (width 0.05))
+    (fp_line (start -1.68 -0.95) (end 1.68 -0.95) (layer F.CrtYd) (width 0.05))
+    (fp_line (start -1.68 0.95) (end -1.68 -0.95) (layer F.CrtYd) (width 0.05))
+    (fp_line (start -0.258578 0.71) (end 0.258578 0.71) (layer F.SilkS) (width 0.12))
+    (fp_line (start -0.258578 -0.71) (end 0.258578 -0.71) (layer F.SilkS) (width 0.12))
+    (fp_line (start 1 0.6) (end -1 0.6) (layer F.Fab) (width 0.1))
+    (fp_line (start 1 -0.6) (end 1 0.6) (layer F.Fab) (width 0.1))
+    (fp_line (start -1 -0.6) (end 1 -0.6) (layer F.Fab) (width 0.1))
+    (fp_line (start -1 0.6) (end -1 -0.6) (layer F.Fab) (width 0.1))
+    (pad 2 smd roundrect (at 0.9375 0 270) (size 0.975 1.4) (layers F.Cu F.Paste F.Mask) (roundrect_rratio 0.25)
+      (net 111 Earth))
+    (pad 1 smd roundrect (at -0.9375 0 270) (size 0.975 1.4) (layers F.Cu F.Paste F.Mask) (roundrect_rratio 0.25)
+      (net 1 +5V))
+    (model ${KISYS3DMOD}/Capacitor_SMD.3dshapes/C_0805_2012Metric.wrl
+      (at (xyz 0 0 0))
+      (scale (xyz 1 1 1))
+      (rotate (xyz 0 0 0))
+    )
+  )
   (module Connector_PinHeader_2.54mm:PinHeader_2x03_P2.54mm_Vertical (layer B.Cu)
     (at 103.505 20.955 270)
     (descr "Through hole straight pin header, 2x03, 2.54mm pitch, double rows")
     (tags "Through hole pin header THT 2x03 2.54mm double row")
-    (fp_text reference " " (at 2.54 -2.54) (layer B.SilkS)
+    (fp_text reference J3 (at 2.54 -2.54) (layer B.SilkS)
       (effects (font (size 1 1) (thickness 0.15)) (justify mirror))
     )
@@
   (segment (start 104.744991 22.128009) (end 104.744991 20.350009) (width 0.25) (layer F.Cu) (net 1))
   (segment (start 104.744991 20.350009) (end 105.537 19.558) (width 0.25) (layer F.Cu) (net 1))
+  (segment (start 70.612 107.95) (end 70.485 107.823) (width 0.5) (layer F.Cu) (net 1))
+  (segment (start 70.612 109.8065) (end 70.612 107.95) (width 0.5) (layer F.Cu) (net 1))
   (segment (start 92.46399 108.543214) (end 92.46399 103.59149) (width 0.25) (layer F.Cu) (net 2))
   (segment (start 92.46399 103.59149) (end 91.313 102.4405) (width 0.25) (layer F.Cu) (net 2))
@@
   (segment (start 103.69302 33.33998) (end 108.585 28.448) (width 0.35) (layer F.Cu) (net 111))
   (segment (start 108.585 23.495) (end 108.585 28.448) (width 0.35) (layer F.Cu) (net 111))
+  (segment (start 69.215 113.566) (end 69.215 113.665) (width 0.5) (layer F.Cu) (net 111))
+  (segment (start 70.612 112.169) (end 69.215 113.566) (width 0.5) (layer F.Cu) (net 111))
+  (segment (start 70.612 111.6815) (end 70.612 112.169) (width 0.5) (layer F.Cu) (net 111))
   (segment (start 103.62999 100.96701) (end 102.927 101.67) (width 0.25) (layer F.Cu) (net 112))
   (segment (start 106.299 98.6305) (end 104.63765 98.6305) (width 0.25) (layer F.Cu) (net 112))

Commit message: joo
Parts:
- removed R41, R42, R43, R44, R45, R46, R47, R48, R49, R50, R51, R52, R53: 1M, Resistor_SMD:R_0805_2012Metric
- removed the REF** at (107.6, 93.7)
- removed the REF** at (108.2, 103.9)
- removed the REF** at (104.1, 92.6)
- removed the REF** at (111.0, 104.0)
- removed the REF** at (102.2, 29.0)
- removed the REF** at (112.6, 101.7)
- added C10: 100n, Capacitor_SMD:C_0805_2012Metric, F.Cu at (115.2, 14.5)
- added C11: 100u, Capacitor_SMD:CP_Elec_6.3x7.7, F.Cu at (99.9, 17.0)
- added J4: Barrel_Jack, Connector_BarrelJack:BarrelJack_Horizontal, F.Cu at (67.1, 101.9)
- added REF**: 0, Resistor_SMD:R_0805_2012Metric, F.Cu at (104.9, 92.0)
- added REF**: 0, Resistor_SMD:R_0805_2012Metric, F.Cu at (111.0, 104.4)
- added REF**: 0, Resistor_SMD:R_0805_2012Metric, F.Cu at (102.2, 31.0)
- added REF**: 0, Resistor_SMD:R_0805_2012Metric, F.Cu at (113.5, 102.4)
- C2: value 100nF -> 100n
- C9: value 100uF -> 100n; footprint Capacitor_SMD:CP_Elec_6.3x7.7 -> Capacitor_SMD:C_0805_2012Metric
- J1: footprint Resistor_SMD:R_1210_3225Metric -> Connector_PinHeader_2.54mm:PinHeader_1x03_P2.54mm_Vertical
- R1: value 47k -> 1k
- moved C2 134.7 mm to (164.8, 14.5), turned to 90 degrees
- moved C9 93.7 mm to (65.9, 14.2), turned to 90 degrees
- moved C4 60.7 mm to (20.8, 82.2), turned to 180 degrees
- moved R92 9.72 mm to (77.2, 91.9), turned to 180 degrees
- moved R39 8.79 mm to (114.7, 105.9), turned to 180 degrees
- moved C6 6.99 mm to (86.6, 91.9), turned to 0 degrees
- moved R90 6.25 mm to (82.0, 91.9), turned to 0 degrees
- moved C7 5.89 mm to (79.1, 103.6), turned to 0 degrees
- moved J1 5.80 mm to (115.7, 96.5), turned to 270 degrees
- moved R31 5.43 mm to (111.5, 19.8)
- moved R32 4.88 mm to (119.8, 18.0), turned to 180 degrees
- moved C5 4.13 mm to (22.9, 14.1), turned to 90 degrees
- moved SW1 3.90 mm to (83.1, 101.6)
- moved SW2 3.90 mm to (74.3, 101.6)
- moved R1 3.84 mm to (110.1, 100.1), turned to 90 degrees
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Connections:
- J1 pad 1: Net-(J1-Pad1) -> +5V
- J1 pad 2: Earth -> Net-(J1-Pad2)
- R1 pad 1: Net-(J1-Pad1) -> Net-(R1-Pad1)
- R1 pad 2: +5V -> Net-(J1-Pad2)
- U1 pad 19: Net-(J1-Pad1) -> Net-(R1-Pad1)
Routing:
- net Earth: track 976.3 -> 942.3 mm
- net /Naytto/Ghi0: track 175.7 -> 207.6 mm
- net /Naytto/Numero/Cat3b: track 306.4 -> 291.3 mm
- net /Naytto/Numero/Cat6a: track 234.4 -> 219.5 mm
- net Net-(J1-Pad1): track 14.5 -> 0.00 mm
- net /Naytto/Numero/Cat5: track 347.4 -> 333.4 mm
- net /Naytto/Glo3: track 200.4 -> 186.8 mm
- net /Naytto/Numero/Cat6b: track 211.3 -> 197.9 mm
- net /Naytto/Numero/Cat4: track 499.7 -> 487.0 mm
- net /Naytto/GloB: track 60.8 -> 48.8 mm
- net /Naytto/Numero/Cat7: track 241.4 -> 229.7 mm
- net Net-(R1-Pad1): track 0.00 -> 10.8 mm
- net Net-(Q32-Pad3): track 9.27 -> 20.0 mm
- net /Naytto/Numero/CatA: track 368.3 -> 358.0 mm
- net /Naytto/Ghi1: track 113.1 -> 103.5 mm, vias 2 -> 0
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
Commit message: nonni
Parts:
- removed the REF** at (104.9, 92.0)
- removed the REF** at (111.0, 104.4)
- removed the REF** at (102.2, 31.0)
- removed the REF** at (113.5, 102.4)
- removed the REF** at (113.5, 100.3)
- added REF**: 0, Resistor_SMD:R_0805_2012Metric, F.Cu at (110.1, 103.8)
- J3: footprint Connector_PinHeader_2.54mm:PinHeader_2x03_P2.54mm_Vertical -> Connector_Molex:Molex_Pico-Clasp_501331-0607_1x06-1MP_P1.00mm_Vertical; moved to F.Cu
- moved R17 67.9 mm to (102.8, 21.8), turned to 180 degrees
- moved J3 65.9 mm to (111.5, 90.0), turned to 0 degrees
- moved R39 17.0 mm to (118.9, 89.4), turned to 90 degrees
- moved R4 11.2 mm to (105.5, 91.9), turned to 270 degrees
- turned Q33 to 90 degrees
Routing:
- net /Naytto/Ghi0: track 207.6 -> 95.6 mm, vias 2 -> 0
- net /Naytto/Glo4: track 120.7 -> 49.9 mm
- net /Naytto/Glo5: track 123.6 -> 53.9 mm
- net /Naytto/Glo3: track 186.8 -> 118.1 mm
- net Net-(Q2-Pad1): track 3.66 -> 72.1 mm, vias 0 -> 2
- net Earth: track 942.3 -> 874.1 mm
- net Net-(J3-Pad5): track 98.8 -> 33.3 mm
- net +5V: track 428.9 -> 406.4 mm
- net Net-(Q32-Pad3): track 20.0 -> 9.34 mm
- net /Naytto/GloB: track 48.8 -> 39.6 mm
- net /Naytto/Ghi1: track 103.5 -> 99.9 mm
- net Net-(Q32-Pad1): track 8.04 -> 6.37 mm
- net /Naytto/sheet5E58E229/Collector: track 47.4 -> 46.8 mm

Commit message: ei niin pahan näköne
Parts:
- removed the REF** at (119.3, 53.3)
- moved R18 62.2 mm to (105.5, 19.7), turned to 270 degrees
- moved Q2 53.5 mm to (114.2, 18.7), turned to 0 degrees
- moved C2 47.6 mm to (117.2, 14.5)
- moved R32 12.5 mm to (107.6, 20.7), turned to 270 degrees
- moved R31 5.97 mm to (106.8, 23.5)
- moved Q3 3.56 mm to (114.2, 22.2)
- moved D3 1.80 mm to (164.5, 21.6), turned to 180 degrees
Routing:
- net Net-(Q2-Pad1): track 72.1 -> 11.2 mm, vias 2 -> 0
- net /Naytto/Numero/Anode: track 204.4 -> 255.5 mm
- net +5V: track 406.4 -> 356.4 mm
- net /Naytto/Ghi1: track 99.9 -> 94.4 mm
- net /Naytto/sheet5E6237CA/Anode: track 229.7 -> 235.0 mm
- net Net-(Q3-Pad1): track 7.12 -> 10.3 mm
- net Net-(D13-Pad2): track 28.8 -> 29.5 mm
- net /Naytto/Numero/Cat3a: track 695.3 -> 695.8 mm, vias 6 -> 8

Commit message: tilasin nää
Parts:
- added C12: 100nF, Capacitor_SMD:C_0805_2012Metric, F.Cu at (56.3, 103.8)
- moved R11 54.8 mm to (139.6, 108.0)
- moved R19 19.6 mm to (115.1, 106.0), turned to 180 degrees
- moved R15 14.0 mm to (115.1, 104.0), turned to 180 degrees
- moved D3 1.80 mm to (163.2, 22.9), turned to 90 degrees
Routing:
- net /Naytto/Glo3: track 118.1 -> 63.0 mm, vias 2 -> 0
- net Net-(Q12-Pad3): track 9.18 -> 62.8 mm
- net /Naytto/Glo5: track 53.9 -> 30.6 mm
- net Net-(Q18-Pad3): track 9.36 -> 29.9 mm
- net /Naytto/Glo4: track 49.9 -> 29.8 mm
- net Net-(Q16-Pad3): track 9.32 -> 24.8 mm
- net /Naytto/Numero/Cat3a: track 695.8 -> 694.5 mm
- net /Naytto/Ghi3: track 148.2 -> 147.4 mm
- net Net-(D13-Pad2): track 29.5 -> 28.8 mm
- net /Naytto/Numero/Anode: track 255.5 -> 255.0 mm
Other:
- outline, holes or cut-outs redrawn
