File: kello-yritys2.sch (KiCad schematic (older format))
At the start: 13 parts, among them J1 Conn_01x02_Male_To_Opto, J2 USB_B_Micro, J3 AVR-ISP-6, Q1 TEPT4400, U1 ATmega328PB-AU

Commit message: joo
Connections:
- net Naytto/Glo0: now also J3.4 (MOSI), U1.15 (PB3); no longer U1.7 (XTAL1/PB6)
- net Naytto/Glo1: now also J3.1 (MISO), U1.16 (PB4); no longer U1.8 (XTAL2/PB7)
- net Naytto/Glo2: now also J3.3 (SCK), U1.17 (PB5); no longer U1.9 (PD5)
- net Naytto/Glo3: now also U1.9 (PD5); no longer U1.10 (PD6)
- net Naytto/Glo4: now also U1.7 (XTAL1/PB6); no longer U1.11 (PD7)
- net Naytto/Glo5: now also U1.8 (XTAL2/PB7); no longer U1.12 (PB0)
- net Naytto/Glo6: now also U1.10 (PD6); no longer U1.13 (PB1)
- net Naytto/Glo7: now also U1.11 (PD7); no longer U1.14 (PB2)
- net Naytto/Glo8: now also U1.13 (PB1); no longer J3.4 (MOSI), U1.15 (PB3)
- net Naytto/Glo9: now also U1.14 (PB2); no longer J3.1 (MISO), U1.16 (PB4)
- net Naytto/GloA: now also U1.12 (PB0); no longer J3.3 (SCK), U1.17 (PB5)
Changed lines of the file:
@@
 $EndComp
-Wire Wire Line
-	3150 2700 4050 2700
-Wire Wire Line
-	3950 2800 3150 2800
-Wire Wire Line
-	3150 2900 3850 2900
 Wire Wire Line
 	3750 3000 3150 3000
@@
 	3150 3200 3550 3200
 Wire Wire Line
-	3150 3300 3250 3300
-Wire Wire Line
-	3250 3300 3250 2500
-Wire Wire Line
-	3350 2600 3350 3400
-Wire Wire Line
-	3350 3400 3150 3400
-Wire Wire Line
-	3150 4900 4150 4900
-Wire Wire Line
-	3150 5000 4250 5000
-Wire Wire Line
-	3150 5100 4350 5100
-Wire Wire Line
 	3450 3600 3150 3600
 Wire Wire Line
-	3350 2600 4900 2600
-Wire Wire Line
-	3250 2500 4900 2500
-Wire Wire Line
-	4150 2700 4900 2700
-Wire Wire Line
-	4150 2700 4150 4900
-Wire Wire Line
-	4900 2800 4250 2800
-Wire Wire Line
-	4250 2800 4250 5000
-Wire Wire Line
-	4350 2900 4900 2900
-Wire Wire Line
-	4350 2900 4350 5100
-Wire Wire Line
-	4050 3000 4900 3000
-Wire Wire Line
-	4050 2700 4050 3000
-Wire Wire Line
-	4900 3100 3950 3100
-Wire Wire Line
-	3950 3100 3950 2800
-Wire Wire Line
-	3850 2900 3850 3200
-Wire Wire Line
-	3850 3200 4900 3200
-Wire Wire Line
-	4900 3300 3750 3300
-Wire Wire Line
-	3750 3300 3750 3000
-Wire Wire Line
-	3650 3100 3650 3400
-Wire Wire Line
-	3650 3400 4900 3400
-Wire Wire Line
-	4900 3500 3550 3500
-Wire Wire Line
-	3550 3500 3550 3200
-Connection ~ 3750 3000
-Connection ~ 3650 3100
-Wire Wire Line
-	4750 1800 4750 4200
-Wire Wire Line
-	3150 4200 4750 4200
+	4750 1800 4750 2300
+Wire Wire Line
+	3150 4200 3950 4200
 Wire Wire Line
 	4750 1600 3750 1600
 Wire Wire Line
-	3750 1600 3750 3000
+	3750 1600 3750 2500
 Wire Wire Line
 	4750 1500 3650 1500
 Wire Wire Line
-	3650 1500 3650 3100
+	3650 1500 3650 2600
 Wire Wire Line
 	4750 1700 3550 1700
 Wire Wire Line
-	3550 1700 3550 3200
-Connection ~ 3550 3200
+	3550 1700 3550 2400
 $Comp
 L Device:R R4
@@
 	3250 1800 3450 1800
 Wire Wire Line
-	3450 1800 3450 3600
-Wire Wire Line
 	3250 2200 3250 2300
 Wire Wire Line
@@
 Wire Wire Line
 	800  2700 800  2800
-Wire Wire Line
-	4050 4800 4050 3600
-Wire Wire Line
-	4050 3600 4900 3600
-Wire Wire Line
-	3150 4800 4050 4800
 Wire Wire Line
 	1500 5750 1500 5700
@@
 Wire Wire Line
 	1200 2700 1600 2700
+Wire Wire Line
+	4800 2700 4900 2700
+Wire Wire Line
+	3150 2700 4650 2700
+Wire Wire Line
+	4900 3600 4800 3600
+Wire Wire Line
+	4800 3600 4800 4800
+Wire Wire Line
+	3150 4800 4800 4800
+Wire Wire Line
+	3750 2500 4900 2500
+Connection ~ 3750 2500
+Wire Wire Line
+	3750 2500 3750 3000
+Connection ~ 3650 2600
+Wire Wire Line
+	3650 2600 3650 3100
+Wire Wire Line
+	3650 2600 4900 2600
+Wire Wire Line
+	3450 1800 3450 3600
+Wire Wire Line
+	4800 2700 4800 2400
+Wire Wire Line
+	4800 2400 3550 2400
+Connection ~ 3550 2400
+Wire Wire Line
+	3550 2400 3550 3200
+Wire Wire Line
+	3150 2900 3850 2900
+Wire Wire Line
+	4250 2800 4250 3300
+Wire Wire Line
+	3150 2800 4250 2800
+Wire Wire Line
+	4250 3300 4900 3300
+Wire Wire Line
+	4900 2800 4350 2800
+Wire Wire Line
+	4350 2800 4350 4900
+Wire Wire Line
+	3150 4900 4350 4900
+Wire Wire Line
+	4900 3100 4450 3100
+Wire Wire Line
+	4450 3100 4450 5000
+Wire Wire Line
+	3150 5000 4450 5000
+Wire Wire Line
+	4550 5100 4550 3200
+Wire Wire Line
+	4550 3200 4900 3200
+Wire Wire Line
+	3150 5100 4550 5100
+Wire Wire Line
+	4650 3500 4650 2700
+Wire Wire Line
+	4650 3500 4900 3500
+Wire Wire Line
+	3850 2900 3850 3400
+Wire Wire Line
+	4150 3000 4900 3000
+Wire Wire Line
+	3150 3400 3750 3400
+Wire Wire Line
+	4050 2900 4900 2900
+Wire Wire Line
+	3150 3300 3650 3300
+Wire Wire Line
+	4750 2300 3950 2300
+Wire Wire Line
+	3950 2300 3950 4200
+Wire Wire Line
+	4050 3100 3750 3100
+Wire Wire Line
+	3750 3100 3750 3200
+Wire Wire Line
+	4050 3100 4050 2900
+Wire Wire Line
+	3750 3200 3650 3200
+Wire Wire Line
+	3650 3200 3650 3300
+Wire Wire Line
+	3750 3400 3750 3300
+Wire Wire Line
+	3750 3300 4150 3300
+Wire Wire Line
+	4150 3300 4150 3000
+Wire Wire Line
+	3850 3400 4900 3400
 $EndSCHEMATC

Commit message: joo
Parts:
- removed C2: 1n, Capacitor_SMD:C_0805_2012Metric, symbol Device:C
- removed R2: 150k, Resistor_SMD:R_0805_2012Metric, symbol Device:R
Connections:
- net +5V: no longer C1.2, C3.2, C8.2, J1.2 (Pin_2), J2.5 (GND), J2.6 (Shield), J3.6 (GND), Q1.2 (E), U1.21 (GND), U1.5 (GND)
- net Naytto/Ghi0: now also U1.31 (PD1); no longer U1.30 (PD0)
- net Naytto/Ghi1: now also U1.32 (PD2); no longer U1.31 (PD1)
- net Naytto/Ghi2: now also U1.1 (PD3); no longer U1.32 (PD2)
- net Naytto/Ghi3: now also U1.2 (PD4); no longer U1.1 (PD3)
- net Naytto/Glo0: now also U1.9 (PD5); no longer J3.4 (MOSI), U1.15 (PB3)
- net Naytto/Glo1: now also U1.8 (XTAL2/PB7); no longer J3.1 (MISO), U1.16 (PB4)
- net Naytto/Glo2: now also U1.7 (XTAL1/PB6); no longer J3.3 (SCK), U1.17 (PB5)
- net Naytto/Glo3: now also J3.4 (MOSI), U1.15 (PB3); no longer U1.9 (PD5)
- net Naytto/Glo4: now also J3.3 (SCK), U1.17 (PB5); no longer U1.7 (XTAL1/PB6)
- net Naytto/Glo5: now also J3.1 (MISO), U1.16 (PB4); no longer U1.8 (XTAL2/PB7)
- net Naytto/Glo6: now also U1.14 (PB2); no longer U1.10 (PD6)
- net Naytto/Glo7: now also U1.13 (PB1); no longer U1.11 (PD7)
- net Naytto/Glo8: now also U1.11 (PD7); no longer U1.13 (PB1)
- net Naytto/Glo9: now also U1.10 (PD6); no longer U1.14 (PB2)
- net Naytto/GloB: now also U1.30 (PD0); no longer U1.2 (PD4)
- net at U1.22 (PE3): no longer J2.2 (D-)
- new net Earth: C1.2, C3.2, C8.2, J1.2 (Pin_2), J2.5 (GND), J2.6 (Shield), J3.6 (GND), Q1.2 (E), U1.21 (GND), U1.5 (GND)
Changed lines of the file:
@@
 $EndDescr
 $Sheet
-S 4900 2400 600  1300
+S 4950 2400 600  1300
 U 5E309501
 F0 "Naytto" 50
 F1 "naytto.sch" 50
-F2 "Glo0" I L 4900 2500 50
-F3 "Glo1" I L 4900 2600 50
-F4 "Glo2" I L 4900 2700 50
-F5 "Glo3" I L 4900 2800 50
-F6 "Glo4" I L 4900 2900 50
-F7 "Glo5" I L 4900 3000 50
-F8 "Glo6" I L 4900 3100 50
-F9 "Glo7" I L 4900 3200 50
-F10 "Glo8" I L 4900 3300 50
-F11 "Glo9" I L 4900 3400 50
-F12 "GloA" I L 4900 3500 50
-F13 "Ghi0" I R 5500 2500 50
-F14 "Ghi1" I R 5500 2600 50
-F15 "Ghi2" I R 5500 2700 50
-F16 "Ghi3" I R 5500 2800 50
-F17 "GloB" I L 4900 3600 50
+F2 "Glo0" I L 4950 2500 50
+F3 "Glo1" I L 4950 2600 50
+F4 "Glo2" I L 4950 2700 50
+F5 "Glo3" I L 4950 2800 50
+F6 "Glo4" I L 4950 2900 50
+F7 "Glo5" I L 4950 3000 50
+F8 "Glo6" I L 4950 3100 50
+F9 "Glo7" I L 4950 3200 50
+F10 "Glo8" I L 4950 3300 50
+F11 "Glo9" I L 4950 3400 50
+F12 "GloA" I L 4950 3500 50
+F13 "Ghi0" I R 5550 2500 50
+F14 "Ghi1" I R 5550 2600 50
+F15 "Ghi2" I R 5550 2700 50
+F16 "Ghi3" I R 5550 2800 50
+F17 "GloB" I L 4950 3600 50
 $EndSheet
 $Comp
@@
 	-1   0    0    -1
 $EndComp
-$Comp
-L MCU_Microchip_ATmega:ATmega328PB-AU U1
-U 1 1 5E7981AC
-P 2550 3900
-F 0 "U1" H 2550 2311 50  0000 C CNN
-F 1 "ATmega328PB-AU" H 2550 2220 50  0000 C CNN
-F 2 "Package_QFP:TQFP-32_7x7mm_P0.8mm" H 2550 3900 50  0001 C CIN
-F 3 "http://ww1.microchip.com/downloads/en/DeviceDoc/40001906C.pdf" H 2550 3900 50  0001 C CNN
-	1    2550 3900
-	1    0    0    -1
-$EndComp
 Wire Wire Line
 	3750 3000 3150 3000
@@
 	4750 1600 3750 1600
 Wire Wire Line
-	3750 1600 3750 2500
-Wire Wire Line
 	4750 1500 3650 1500
 Wire Wire Line
-	3650 1500 3650 2600
-Wire Wire Line
 	4750 1700 3550 1700
-Wire Wire Line
-	3550 1700 3550 2400
 $Comp
 L Device:R R4
@@
 Wire Wire Line
 	5250 2100 5250 2200
-Wire Wire Line
-	3150 4400 5600 4400
-Wire Wire Line
-	5600 4400 5600 2500
-Wire Wire Line
-	5600 2500 5500 2500
-Wire Wire Line
-	5500 2600 5700 2600
-Wire Wire Line
-	5700 2600 5700 4500
-Wire Wire Line
-	5700 4500 3150 4500
-Wire Wire Line
-	3150 4600 5800 4600
-Wire Wire Line
-	5800 4600 5800 2700
-Wire Wire Line
-	5800 2700 5500 2700
-Wire Wire Line
-	5500 2800 5900 2800
-Wire Wire Line
-	5900 2800 5900 4700
-Wire Wire Line
-	5900 4700 3150 4700
 $Comp
 L power:+5V #PWR0105
@@
 	1    0    0    -1
 $EndComp
-Wire Wire Line
-	2550 5700 2550 5400
 $Comp
 L Device:R R1
@@
 $EndComp
 $Comp
-L Device:C C2
-U 1 1 5E83BA1A
-P 1500 5500
-F 0 "C2" H 1615 5546 50  0000 L CNN
-F 1 "1n" H 1615 5455 50  0000 L CNN
-F 2 "Capacitor_SMD:C_0805_2012Metric" H 1538 5350 50  0001 C CNN
-F 3 "~" H 1500 5500 50  0001 C CNN
-	1    1500 5500
-	1    0    0    -1
-$EndComp
-$Comp
 L Connector:Conn_01x02_Male J1
 U 1 1 5E849348
@@
 Wire Wire Line
 	1500 5750 1500 5700
-Connection ~ 1500 5700
-Wire Wire Line
-	1500 5700 1500 5650
 Wire Wire Line
 	750  5700 1500 5700
@@
 	1450 4300 1450 4500
 Wire Wire Line
-	1450 4500 1950 4500
-Wire Wire Line
 	750  5600 1350 5600
 Wire Wire Line
 	1950 4600 1350 4600
-Wire Wire Line
-	1350 4600 1350 5300
-Wire Wire Line
-	1350 5300 1500 5300
-Wire Wire Line
-	1500 5300 1500 5350
-Connection ~ 1350 5300
-Wire Wire Line
-	1350 5300 1350 5600
-Wire Wire Line
-	1500 5300 1500 5250
-Connection ~ 1500 5300
 Wire Wire Line
 	1500 4950 1500 4850
@@
 $EndComp
 $Comp
-L Device:R R2
-U 1 1 5EA08B4B
-P 1500 6450
-F 0 "R2" V 1293 6450 50  0000 C CNN
-F 1 "150k" V 1384 6450 50  0000 C CNN
-F 2 "Resistor_SMD:R_0805_2012Metric" V 1430 6450 50  0001 C CNN
-F 3 "~" H 1500 6450 50  0001 C CNN
-	1    1500 6450
-	0    1    1    0
-$EndComp
-Wire Wire Line
-	1350 6450 1250 6450
-Wire Wire Line
-	1650 6450 1750 6450
-Wire Wire Line
-	1750 6450 1750 6250
-Wire Wire Line
-	1750 6250 1350 6250
-Connection ~ 1350 6250
-Wire Wire Line
-	1250 6550 1950 6550
-Wire Wire Line
-	1950 6550 1950 4700
-$Comp
 L Device:C C8
 U 1 1 5E47CB5F
@@
 Connection ~ 1600 1700
 Wire Wire Line
-	1950 2700 1600 2700
-Connection ~ 1950 2700
-Wire Wire Line
 	800  2700 1200 2700
-Connection ~ 1600 2700
 Wire Wire Line
 	1200 2350 1200 2700
@@
 	1200 2700 1600 2700
 Wire Wire Line
-	4800 2700 4900 2700
-Wire Wire Line
-	3150 2700 4650 2700
-Wire Wire Line
-	4900 3600 4800 3600
-Wire Wire Line
-	4800 3600 4800 4800
-Wire Wire Line
-	3150 4800 4800 4800
-Wire Wire Line
-	3750 2500 4900 2500
-Connection ~ 3750 2500
-Wire Wire Line
-	3750 2500 3750 3000
-Connection ~ 3650 2600
-Wire Wire Line
-	3650 2600 3650 3100
-Wire Wire Line
-	3650 2600 4900 2600
-Wire Wire Line
 	3450 1800 3450 3600
 Wire Wire Line
-	4800 2700 4800 2400
-Wire Wire Line
-	4800 2400 3550 2400
-Connection ~ 3550 2400
-Wire Wire Line
-	3550 2400 3550 3200
-Wire Wire Line
-	3150 2900 3850 2900
-Wire Wire Line
-	4250 2800 4250 3300
-Wire Wire Line
-	3150 2800 4250 2800
-Wire Wire Line
-	4250 3300 4900 3300
-Wire Wire Line
-	4900 2800 4350 2800
-Wire Wire Line
-	4350 2800 4350 4900
-Wire Wire Line
-	3150 4900 4350 4900
-Wire Wire Line
-	4900 3100 4450 3100
-Wire Wire Line
-	4450 3100 4450 5000
-Wire Wire Line
-	3150 5000 4450 5000
-Wire Wire Line
-	4550 5100 4550 3200
-Wire Wire Line
-	4550 3200 4900 3200
-Wire Wire Line
-	3150 5100 4550 5100
-Wire Wire Line
-	4650 3500 4650 2700
-Wire Wire Line
-	4650 3500 4900 3500
-Wire Wire Line
-	3850 2900 3850 3400
-Wire Wire Line
-	4150 3000 4900 3000
-Wire Wire Line
-	3150 3400 3750 3400
-Wire Wire Line
-	4050 2900 4900 2900
-Wire Wire Line
-	3150 3300 3650 3300
-Wire Wire Line
 	4750 2300 3950 2300
 Wire Wire Line
 	3950 2300 3950 4200
 Wire Wire Line
-	4050 3100 3750 3100
-Wire Wire Line
-	3750 3100 3750 3200
-Wire Wire Line
-	4050 3100 4050 2900
-Wire Wire Line
-	3750 3200 3650 3200
-Wire Wire Line
-	3650 3200 3650 3300
-Wire Wire Line
-	3750 3400 3750 3300
-Wire Wire Line
-	3750 3300 4150 3300
-Wire Wire Line
-	4150 3300 4150 3000
-Wire Wire Line
-	3850 3400 4900 3400
+	3650 1500 3650 3100
+Wire Wire Line
+	3750 1600 3750 2600
+Wire Wire Line
+	3550 1700 3550 3200
+Wire Wire Line
+	5650 2500 5550 2500
+Wire Wire Line
+	5550 2600 5750 2600
+Wire Wire Line
+	5850 2700 5550 2700
+Wire Wire Line
+	5550 2800 5950 2800
+Wire Wire Line
+	3150 2700 3250 2700
+Wire Wire Line
+	4150 2900 4150 3100
+Wire Wire Line
+	4150 3100 4950 3100
+Wire Wire Line
+	3150 2900 4150 2900
+Connection ~ 3650 3100
+Connection ~ 3550 3200
+Wire Wire Line
+	3150 2800 4350 2800
+Wire Wire Line
+	3550 3200 4250 3200
+Connection ~ 3750 2600
+Wire Wire Line
+	3750 2600 3750 3000
+Wire Wire Line
+	3850 3100 3850 3000
+Wire Wire Line
+	3650 3100 3850 3100
+Wire Wire Line
+	3850 3000 4950 3000
+Wire Wire Line
+	3150 3400 4650 3400
+Wire Wire Line
+	4250 2900 4250 3200
+Wire Wire Line
+	4250 2900 4950 2900
+Wire Wire Line
+	4350 3200 4350 2800
+Wire Wire Line
+	4350 3200 4950 3200
+Wire Wire Line
+	4450 2800 4450 2600
+Wire Wire Line
+	4450 2600 3750 2600
+Wire Wire Line
+	4450 2800 4950 2800
+Wire Wire Line
+	4950 3600 4850 3600
+Wire Wire Line
+	4950 2500 4550 2500
+Wire Wire Line
+	4550 2500 4550 4900
+Wire Wire Line
+	3150 4900 4550 4900
+Wire Wire Line
+	4650 2600 4650 3400
+Wire Wire Line
+	4650 2600 4950 2600
+Wire Wire Line
+	3150 5100 4150 5100
+Wire Wire Line
+	3250 3500 3250 2700
+Wire Wire Line
+	3250 3500 4950 3500
+Wire Wire Line
+	4050 2700 4050 3300
+Wire Wire Line
+	4050 2700 4950 2700
+Wire Wire Line
+	4150 3300 4150 5100
+Wire Wire Line
+	4150 3300 4950 3300
+Wire Wire Line
+	4950 3400 4750 3400
+Wire Wire Line
+	4750 3400 4750 5000
+Wire Wire Line
+	3150 5000 4750 5000
+Wire Wire Line
+	3150 3300 4050 3300
+Wire Wire Line
+	1450 4500 1950 4500
+$Comp
+L MCU_Microchip_ATmega:ATmega328PB-AU U1
+U 1 1 5E7981AC
+P 2550 3900
+F 0 "U1" H 2550 2311 50  0000 C CNN
+F 1 "ATmega328PB-AU" H 2550 2220 50  0000 C CNN
+F 2 "Package_QFP:TQFP-32_7x7mm_P0.8mm" H 2550 3900 50  0001 C CIN
+F 3 "http://ww1.microchip.com/downloads/en/DeviceDoc/40001906C.pdf" H 2550 3900 50  0001 C CNN
+	1    2550 3900
+	1    0    0    -1
+$EndComp
+Wire Wire Line
+	4850 3600 4850 4400
+Wire Wire Line
+	4850 4400 3150 4400
+Wire Wire Line
+	5950 2800 5950 4800
+Wire Wire Line
+	3150 4800 5950 4800
+Wire Wire Line
+	5850 4700 3150 4700
+Wire Wire Line
+	5850 2700 5850 4700
+Wire Wire Line
+	3150 4600 5750 4600
+Wire Wire Line
+	5750 2600 5750 4600
+Wire Wire Line
+	3150 4500 5650 4500
+Wire Wire Line
+	5650 2500 5650 4500
+Wire Wire Line
+	2550 5400 2550 5700
+Wire Wire Line
+	1350 4600 1350 5600
+Wire Wire Line
+	1500 5600 1350 5600
+Wire Wire Line
+	1500 5250 1500 5600
+Connection ~ 1350 5600
+$Comp
+L power:Earth #PWR?
+U 1 1 5EB8854D
+P 4450 5850
+F 0 "#PWR?" H 4450 5600 50  0001 C CNN
+F 1 "Earth" H 4450 5700 50  0001 C CNN
+F 2 "" H 4450 5850 50  0001 C CNN
+F 3 "~" H 4450 5850 50  0001 C CNN
+	1    4450 5850
+	1    0    0    -1
+$EndComp
+$Comp
+L power:GNDREF #PWR?
+U 1 1 5EB889B1
+P 4650 5850
+F 0 "#PWR?" H 4650 5600 50  0001 C CNN
+F 1 "GNDREF" H 4655 5677 50  0000 C CNN
+F 2 "" H 4650 5850 50  0001 C CNN
+F 3 "" H 4650 5850 50  0001 C CNN
+	1    4650 5850
+	1    0    0    -1
+$EndComp
+Wire Wire Line
+	4650 5850 4450 5850
 $EndSCHEMATC

Commit message: joo
Connections:
- net Naytto/Ghi0: now also U1.32 (PD2); no longer U1.31 (PD1)
- net Naytto/Ghi1: now also U1.31 (PD1); no longer U1.32 (PD2)
Changed lines of the file:
@@
 	3550 1700 3550 3200
-Wire Wire Line
-	5650 2500 5550 2500
-Wire Wire Line
-	5550 2600 5750 2600
 Wire Wire Line
 	5850 2700 5550 2700
@@
 	3150 4600 5750 4600
 Wire Wire Line
-	5750 2600 5750 4600
-Wire Wire Line
 	3150 4500 5650 4500
-Wire Wire Line
-	5650 2500 5650 4500
 Wire Wire Line
 	2550 5400 2550 5700
@@
 Connection ~ 1350 5600
 $Comp
-L power:Earth #PWR?
+L power:Earth #PWR0119
 U 1 1 5EB8854D
 P 4450 5850
-F 0 "#PWR?" H 4450 5600 50  0001 C CNN
+F 0 "#PWR0119" H 4450 5600 50  0001 C CNN
 F 1 "Earth" H 4450 5700 50  0001 C CNN
 F 2 "" H 4450 5850 50  0001 C CNN
@@
 $EndComp
 $Comp
-L power:GNDREF #PWR?
+L power:GNDREF #PWR0120
 U 1 1 5EB889B1
 P 4650 5850
-F 0 "#PWR?" H 4650 5600 50  0001 C CNN
+F 0 "#PWR0120" H 4650 5600 50  0001 C CNN
 F 1 "GNDREF" H 4655 5677 50  0000 C CNN
 F 2 "" H 4650 5850 50  0001 C CNN
@@
 Wire Wire Line
 	4650 5850 4450 5850
+Wire Wire Line
+	5550 2600 5650 2600
+Wire Wire Line
+	5650 2600 5650 4500
+Wire Wire Line
+	5550 2500 5750 2500
+Wire Wire Line
+	5750 2500 5750 4600
 $EndSCHEMATC

Commit message: joo
Parts:
- added R2: 1M, Resistor_SMD:R_0805_2012Metric, symbol Device:R
- Q1: footprint LED_THT:LED_D3.0mm_Clear -> LED_THT:LED_D3.0mm_Front
Connections:
- net +5V: now also R2.1
- net Earth: now also R2.2
Changed lines of the file:
@@
 F 0 "Q1" H 3340 2046 50  0000 L CNN
 F 1 "TEPT4400" H 3340 1955 50  0000 L CNN
-F 2 "LED_THT:LED_D3.0mm_Clear" H 3630 1860 50  0001 C CNN
+F 2 "LED_THT:LED_D3.0mm_Front" H 3630 1860 50  0001 C CNN
 F 3 "https://www.vishay.com/docs/81341/tept4400.pdf" H 3150 2000 50  0001 C CNN
 	1    3150 2000
@@
 Wire Wire Line
 	5750 2500 5750 4600
+$Comp
+L Device:R R2
+U 1 1 5EBF7F26
+P 550 2200
+F 0 "R2" H 620 2246 50  0000 L CNN
+F 1 "1M" H 620 2155 50  0000 L CNN
+F 2 "Resistor_SMD:R_0805_2012Metric" V 480 2200 50  0001 C CNN
+F 3 "~" H 550 2200 50  0001 C CNN
+	1    550  2200
+	1    0    0    -1
+$EndComp
+Wire Wire Line
+	550  2050 550  1700
+Wire Wire Line
+	550  1700 800  1700
+Connection ~ 800  1700
+Wire Wire Line
+	550  2350 550  2700
+Wire Wire Line
+	550  2700 800  2700
 $EndSCHEMATC

Commit message: joo
Parts:
- removed R2: 1M, Resistor_SMD:R_0805_2012Metric, symbol Device:R
Changed lines of the file:
@@
 Wire Wire Line
 	5750 2500 5750 4600
-$Comp
-L Device:R R2
-U 1 1 5EBF7F26
-P 550 2200
-F 0 "R2" H 620 2246 50  0000 L CNN
-F 1 "1M" H 620 2155 50  0000 L CNN
-F 2 "Resistor_SMD:R_0805_2012Metric" V 480 2200 50  0001 C CNN
-F 3 "~" H 550 2200 50  0001 C CNN
-	1    550  2200
-	1    0    0    -1
-$EndComp
-Wire Wire Line
-	550  2050 550  1700
-Wire Wire Line
-	550  1700 800  1700
-Connection ~ 800  1700
-Wire Wire Line
-	550  2350 550  2700
-Wire Wire Line
-	550  2700 800  2700
 $EndSCHEMATC

Commit message: joo
Parts:
- added C2: 100nF, Capacitor_SMD:C_0805_2012Metric, symbol Device:C
- added C9: 100uF, Capacitor_SMD:CP_Elec_6.3x7.7, symbol Device:CP
Connections:
- net +5V: now also C2.1, C9.1
- net Earth: now also C2.2, C9.2
Changed lines of the file:
@@
 Wire Wire Line
 	5750 2500 5750 4600
+$Comp
+L Device:CP C9
+U 1 1 5EDC347B
+P 400 2200
+F 0 "C9" H 518 2246 50  0000 L CNN
+F 1 "100uF" H 518 2155 50  0000 L CNN
+F 2 "Capacitor_SMD:CP_Elec_6.3x7.7" H 438 2050 50  0001 C CNN
+F 3 "~" H 400 2200 50  0001 C CNN
+	1    400  2200
+	1    0    0    -1
+$EndComp
+$Comp
+L Device:C C2
+U 1 1 5EDC38E1
+P 100 2200
+F 0 "C2" H 215 2246 50  0000 L CNN
+F 1 "100nF" H 215 2155 50  0000 L CNN
+F 2 "Capacitor_SMD:C_0805_2012Metric" H 138 2050 50  0001 C CNN
+F 3 "~" H 100 2200 50  0001 C CNN
+	1    100  2200
+	1    0    0    -1
+$EndComp
+Wire Wire Line
+	100  1700 100  2050
+Connection ~ 800  1700
+Wire Wire Line
+	100  2350 100  2700
+Wire Wire Line
+	400  2350 400  2700
+Wire Wire Line
+	100  2700 400  2700
+Wire Wire Line
+	400  2700 800  2700
+Connection ~ 400  2700
+Wire Wire Line
+	400  2050 400  1700
+Wire Wire Line
+	800  1700 400  1700
+Wire Wire Line
+	400  1700 100  1700
+Connection ~ 400  1700
 $EndSCHEMATC
