File: kello-yritys2.sch (KiCad schematic (older format))
At the start: 13 parts, among them J1 Conn_01x02_Male_To_Opto, J2 USB_B_Micro, J3 AVR-ISP-6, Q1 TEPT4400, U1 ATmega328PB-AU

Commit message: joo
Parts:
- removed C2: 100nF, Capacitor_SMD:C_0805_2012Metric, symbol Device:C
- removed C9: 100uF, Capacitor_SMD:CP_Elec_6.3x7.7, symbol Device:CP
- added J4: Barrel_Jack, Connector_BarrelJack:BarrelJack_Horizontal, symbol Connector:Barrel_Jack
- J1: footprint Resistor_SMD:R_1210_3225Metric -> Connector_PinHeader_2.54mm:PinHeader_1x03_P2.54mm_Vertical; symbol Connector:Conn_01x02_Male -> Connector:Conn_01x03_Male
- J3: symbol Connector:AVR-ISP-6 -> kello-yritys2-rescue:AVR-ISP-6-Connector
- R1: value 47k -> 1k
- U1: symbol MCU_Microchip_ATmega:ATmega328PB-AU -> kello-yritys2-rescue:ATmega328PB-AU-MCU_Microchip_ATmega
Connections:
- net +5V: now also J1.1 (Pin_1), J4.1; no longer R1.2
- net Earth: now also J1.3 (Pin_3), J4.2; no longer J1.2 (Pin_2)
- net at R1.1, U1.19 (PE2): no longer J1.1 (Pin_1)
- new net: J1.2 (Pin_2), R1.2
Changed lines of the file:
@@
 $EndComp
 $Comp
-L Connector:AVR-ISP-6 J3
+L kello-yritys2-rescue:AVR-ISP-6-Connector J3
 U 1 1 5E7979B3
 P 5150 1700
@@
 $EndComp
 $Comp
-L Device:R R1
-U 1 1 5E83AA86
-P 1500 5100
-F 0 "R1" V 1293 5100 50  0000 C CNN
-F 1 "47k" V 1384 5100 50  0000 C CNN
-F 2 "Resistor_SMD:R_0805_2012Metric" V 1430 5100 50  0001 C CNN
-F 3 "~" H 1500 5100 50  0001 C CNN
-	1    1500 5100
-	-1   0    0    1
-$EndComp
-$Comp
-L Connector:Conn_01x02_Male J1
+L Connector:Conn_01x03_Male J1
 U 1 1 5E849348
 P 550 5600
 F 0 "J1" H 658 5781 50  0000 C CNN
 F 1 "Conn_01x02_Male_To_Opto" H 658 5690 50  0000 C CNN
-F 2 "Resistor_SMD:R_1210_3225Metric" H 550 5600 50  0001 C CNN
+F 2 "Connector_PinHeader_2.54mm:PinHeader_1x03_P2.54mm_Vertical" H 550 5600 50  0001 C CNN
 F 3 "~" H 550 5600 50  0001 C CNN
 	1    550  5600
@@
 	800  2700 800  2800
 Wire Wire Line
-	1500 5750 1500 5700
-Wire Wire Line
-	750  5700 1500 5700
-$Comp
-L power:+5V #PWR0108
-U 1 1 5E988C60
-P 1500 4850
-F 0 "#PWR0108" H 1500 4700 50  0001 C CNN
-F 1 "+5V" H 1515 5023 50  0000 C CNN
-F 2 "" H 1500 4850 50  0001 C CNN
-F 3 "" H 1500 4850 50  0001 C CNN
-	1    1500 4850
-	1    0    0    -1
-$EndComp
-Wire Wire Line
 	1550 3900 1400 3900
 Wire Wire Line
@@
 Wire Wire Line
 	750  5600 1350 5600
-Wire Wire Line
-	1950 4600 1350 4600
-Wire Wire Line
-	1500 4950 1500 4850
 Wire Wire Line
 	950  6900 950  6850
@@
 L power:Earth #PWR0111
 U 1 1 5E83C367
-P 1500 5750
-F 0 "#PWR0111" H 1500 5500 50  0001 C CNN
-F 1 "Earth" H 1500 5600 50  0001 C CNN
-F 2 "" H 1500 5750 50  0001 C CNN
-F 3 "~" H 1500 5750 50  0001 C CNN
-	1    1500 5750
+P 750 5750
+F 0 "#PWR0111" H 750 5500 50  0001 C CNN
+F 1 "Earth" H 750 5600 50  0001 C CNN
+F 2 "" H 750 5750 50  0001 C CNN
+F 3 "~" H 750 5750 50  0001 C CNN
+	1    750  5750
 	1    0    0    -1
 $EndComp
@@
 	1450 4500 1950 4500
 $Comp
-L MCU_Microchip_ATmega:ATmega328PB-AU U1
+L kello-yritys2-rescue:ATmega328PB-AU-MCU_Microchip_ATmega U1
 U 1 1 5E7981AC
 P 2550 3900
@@
 Wire Wire Line
 	1350 4600 1350 5600
-Wire Wire Line
-	1500 5600 1350 5600
-Wire Wire Line
-	1500 5250 1500 5600
-Connection ~ 1350 5600
 $Comp
 L power:Earth #PWR0119
@@
 	5750 2500 5750 4600
 $Comp
-L Device:CP C9
-U 1 1 5EDC347B
-P 400 2200
-F 0 "C9" H 518 2246 50  0000 L CNN
-F 1 "100uF" H 518 2155 50  0000 L CNN
-F 2 "Capacitor_SMD:CP_Elec_6.3x7.7" H 438 2050 50  0001 C CNN
-F 3 "~" H 400 2200 50  0001 C CNN
-	1    400  2200
-	1    0    0    -1
-$EndComp
-$Comp
-L Device:C C2
-U 1 1 5EDC38E1
-P 100 2200
-F 0 "C2" H 215 2246 50  0000 L CNN
-F 1 "100nF" H 215 2155 50  0000 L CNN
-F 2 "Capacitor_SMD:C_0805_2012Metric" H 138 2050 50  0001 C CNN
-F 3 "~" H 100 2200 50  0001 C CNN
-	1    100  2200
-	1    0    0    -1
-$EndComp
-Wire Wire Line
-	100  1700 100  2050
-Connection ~ 800  1700
-Wire Wire Line
-	100  2350 100  2700
-Wire Wire Line
-	400  2350 400  2700
-Wire Wire Line
-	100  2700 400  2700
-Wire Wire Line
-	400  2700 800  2700
-Connection ~ 400  2700
-Wire Wire Line
-	400  2050 400  1700
-Wire Wire Line
-	800  1700 400  1700
-Wire Wire Line
-	400  1700 100  1700
-Connection ~ 400  1700
+L power:+5V #PWR0108
+U 1 1 5E988C60
+P 750 5250
+F 0 "#PWR0108" H 750 5100 50  0001 C CNN
+F 1 "+5V" H 765 5423 50  0000 C CNN
+F 2 "" H 750 5250 50  0001 C CNN
+F 3 "" H 750 5250 50  0001 C CNN
+	1    750  5250
+	1    0    0    -1
+$EndComp
+Wire Wire Line
+	750  5250 750  5500
+Wire Wire Line
+	750  5700 750  5750
+Wire Wire Line
+	1350 6250 2350 6250
+Wire Wire Line
+	2350 6250 2350 6400
+Wire Wire Line
+	2350 6400 2250 6400
+Connection ~ 1350 6250
+Wire Wire Line
+	2250 6600 2350 6600
+Wire Wire Line
+	2350 6600 2350 6900
+Wire Wire Line
+	2350 6900 950  6900
+$Comp
+L Connector:Barrel_Jack J4
+U 1 1 5EE7A642
+P 1950 6500
+F 0 "J4" H 2007 6825 50  0000 C CNN
+F 1 "Barrel_Jack" H 2007 6734 50  0000 C CNN
+F 2 "Connector_BarrelJack:BarrelJack_Horizontal" H 2000 6460 50  0001 C CNN
+F 3 "~" H 2000 6460 50  0001 C CNN
+	1    1950 6500
+	1    0    0    -1
+$EndComp
+$Comp
+L Device:R R1
+U 1 1 5F38009E
+P 1600 4600
+F 0 "R1" H 1670 4646 50  0000 L CNN
+F 1 "1k" H 1670 4555 50  0000 L CNN
+F 2 "Resistor_SMD:R_0805_2012Metric" V 1530 4600 50  0001 C CNN
+F 3 "~" H 1600 4600 50  0001 C CNN
+	1    1600 4600
+	0    1    1    0
+$EndComp
+Wire Wire Line
+	1350 4600 1450 4600
+Wire Wire Line
+	1750 4600 1950 4600
 $EndSCHEMATC
