File: kello-yritys2.sch (KiCad schematic (older format))
At the start: 12 parts, among them J1 Conn_01x02_Male_To_Opto, J2 USB_B_Micro, J3 AVR-ISP-6, J4 Barrel_Jack, Q1 TEPT4400, U1 ATmega328PB-AU

Commit message: nonni
Parts:
- J3: footprint Connector_PinHeader_2.54mm:PinHeader_2x03_P2.54mm_Vertical -> Connector_Molex:Molex_Pico-Clasp_501331-0607_1x06-1MP_P1.00mm_Vertical
Changed lines of the file:
@@
 F 0 "J3" H 4870 1796 50  0000 R CNN
 F 1 "AVR-ISP-6" H 4870 1705 50  0000 R CNN
-F 2 "Connector_PinHeader_2.54mm:PinHeader_2x03_P2.54mm_Vertical" V 4900 1750 50  0001 C CNN
+F 2 "Connector_Molex:Molex_Pico-Clasp_501331-0607_1x06-1MP_P1.00mm_Vertical" V 4900 1750 50  0000 C CNN
 F 3 " ~" H 3875 1150 50  0001 C CNN
 	1    5150 1700

Commit message: tilasin nää
Parts:
- added C12: 100nF, Capacitor_SMD:C_0805_2012Metric, symbol Device:C
Connections:
- net +5V: now also C12.1
- net Earth: now also C12.2
Changed lines of the file:
@@
 Wire Wire Line
 	1750 4600 1950 4600
+$Comp
+L Device:C C12
+U 1 1 5F4C1EB9
+P 300 2200
+F 0 "C12" H 415 2246 50  0000 L CNN
+F 1 "100nF" H 415 2155 50  0000 L CNN
+F 2 "Capacitor_SMD:C_0805_2012Metric" H 338 2050 50  0001 C CNN
+F 3 "~" H 300 2200 50  0001 C CNN
+	1    300  2200
+	1    0    0    -1
+$EndComp
+Wire Wire Line
+	300  2050 300  1700
+Wire Wire Line
+	300  1700 800  1700
+Connection ~ 800  1700
+Wire Wire Line
+	800  2700 300  2700
+Wire Wire Line
+	300  2700 300  2350
 $EndSCHEMATC
