File: numero.sch (KiCad schematic (older format))
At the start: 20 parts

Commit message: joo
Parts:
- D10, D11, D12, D13, D14, D15, D16, D17, D18, D19, D20, D21, D22, D3, D4, D5, D6, D7, D8, D9: footprint LED_THT:LED_D3.0mm_Clear -> LED_THT:LED_D3.0mm_Front
Changed lines of the file:
@@
 $Descr A4 11693 8268
 encoding utf-8
-Sheet 3 22
+Sheet 18 22
 Title ""
 Date ""
@@
 AR Path="/5E309501/5E62C9E3/5E30964F" Ref="D50"  Part="1"
 AR Path="/5E309501/5E6352C9/5E30964F" Ref="D70"  Part="1"
-F 0 "D10" H 1700 695 50  0000 C CNN
+F 0 "D30" H 1700 695 50  0000 C CNN
 F 1 "LED_Small_ALT" H 1700 786 50  0000 C CNN
-F 2 "LED_THT:LED_D3.0mm_Clear" V 1700 900 50  0001 C CNN
+F 2 "LED_THT:LED_D3.0mm_Front" V 1700 900 50  0001 C CNN
 F 3 "~" V 1700 900 50  0001 C CNN
 	1    1700 900
@@
 AR Path="/5E309501/5E62C9E3/5E3126CB" Ref="D51"  Part="1"
 AR Path="/5E309501/5E6352C9/5E3126CB" Ref="D71"  Part="1"
-F 0 "D11" H 1700 1045 50  0000 C CNN
+F 0 "D31" H 1700 1045 50  0000 C CNN
 F 1 "LED_Small_ALT" H 1700 1136 50  0000 C CNN
-F 2 "LED_THT:LED_D3.0mm_Clear" V 1700 1250 50  0001 C CNN
+F 2 "LED_THT:LED_D3.0mm_Front" V 1700 1250 50  0001 C CNN
 F 3 "~" V 1700 1250 50  0001 C CNN
 	1    1700 1250
@@
 AR Path="/5E309501/5E62C9E3/5E3131D5" Ref="D53"  Part="1"
 AR Path="/5E309501/5E6352C9/5E3131D5" Ref="D73"  Part="1"
-F 0 "D13" H 1700 1845 50  0000 C CNN
+F 0 "D33" H 1700 1845 50  0000 C CNN
 F 1 "LED_Small_ALT" H 1700 1936 50  0000 C CNN
-F 2 "LED_THT:LED_D3.0mm_Clear" V 1700 2050 50  0001 C CNN
+F 2 "LED_THT:LED_D3.0mm_Front" V 1700 2050 50  0001 C CNN
 F 3 "~" V 1700 2050 50  0001 C CNN
 	1    1700 2050
@@
 AR Path="/5E309501/5E62C9E3/5E314557" Ref="D43"  Part="1"
 AR Path="/5E309501/5E6352C9/5E314557" Ref="D63"  Part="1"
-F 0 "D3" H 1150 1845 50  0000 C CNN
+F 0 "D23" H 1150 1845 50  0000 C CNN
 F 1 "LED_Small_ALT" H 1150 1936 50  0000 C CNN
-F 2 "LED_THT:LED_D3.0mm_Clear" V 1150 2050 50  0001 C CNN
+F 2 "LED_THT:LED_D3.0mm_Front" V 1150 2050 50  0001 C CNN
 F 3 "~" V 1150 2050 50  0001 C CNN
 	1    1150 2050
@@
 AR Path="/5E309501/5E62C9E3/5E31CE52" Ref="D54"  Part="1"
 AR Path="/5E309501/5E6352C9/5E31CE52" Ref="D74"  Part="1"
-F 0 "D14" H 1700 2145 50  0000 C CNN
+F 0 "D34" H 1700 2145 50  0000 C CNN
 F 1 "LED_Small_ALT" H 1700 2236 50  0000 C CNN
-F 2 "LED_THT:LED_D3.0mm_Clear" V 1700 2350 50  0001 C CNN
+F 2 "LED_THT:LED_D3.0mm_Front" V 1700 2350 50  0001 C CNN
 F 3 "~" V 1700 2350 50  0001 C CNN
 	1    1700 2350
@@
 AR Path="/5E309501/5E62C9E3/5E31F6AD" Ref="D55"  Part="1"
 AR Path="/5E309501/5E6352C9/5E31F6AD" Ref="D75"  Part="1"
-F 0 "D15" H 1700 2445 50  0000 C CNN
+F 0 "D35" H 1700 2445 50  0000 C CNN
 F 1 "LED_Small_ALT" H 1700 2536 50  0000 C CNN
-F 2 "LED_THT:LED_D3.0mm_Clear" V 1700 2650 50  0001 C CNN
+F 2 "LED_THT:LED_D3.0mm_Front" V 1700 2650 50  0001 C CNN
 F 3 "~" V 1700 2650 50  0001 C CNN
 	1    1700 2650
@@
 AR Path="/5E309501/5E62C9E3/5E31F6C1" Ref="D44"  Part="1"
 AR Path="/5E309501/5E6352C9/5E31F6C1" Ref="D64"  Part="1"
-F 0 "D4" H 1150 2445 50  0000 C CNN
+F 0 "D24" H 1150 2445 50  0000 C CNN
 F 1 "LED_Small_ALT" H 1150 2536 50  0000 C CNN
-F 2 "LED_THT:LED_D3.0mm_Clear" V 1150 2650 50  0001 C CNN
+F 2 "LED_THT:LED_D3.0mm_Front" V 1150 2650 50  0001 C CNN
 F 3 "~" V 1150 2650 50  0001 C CNN
 	1    1150 2650
@@
 AR Path="/5E309501/5E62C9E3/5E323EBF" Ref="D56"  Part="1"
 AR Path="/5E309501/5E6352C9/5E323EBF" Ref="D76"  Part="1"
-F 0 "D16" H 1700 2745 50  0000 C CNN
+F 0 "D36" H 1700 2745 50  0000 C CNN
 F 1 "LED_Small_ALT" H 1700 2836 50  0000 C CNN
-F 2 "LED_THT:LED_D3.0mm_Clear" V 1700 2950 50  0001 C CNN
+F 2 "LED_THT:LED_D3.0mm_Front" V 1700 2950 50  0001 C CNN
 F 3 "~" V 1700 2950 50  0001 C CNN
 	1    1700 2950
@@
 AR Path="/5E309501/5E62C9E3/5E323ED3" Ref="D45"  Part="1"
 AR Path="/5E309501/5E6352C9/5E323ED3" Ref="D65"  Part="1"
-F 0 "D5" H 1150 2745 50  0000 C CNN
+F 0 "D25" H 1150 2745 50  0000 C CNN
 F 1 "LED_Small_ALT" H 1150 2836 50  0000 C CNN
-F 2 "LED_THT:LED_D3.0mm_Clear" V 1150 2950 50  0001 C CNN
+F 2 "LED_THT:LED_D3.0mm_Front" V 1150 2950 50  0001 C CNN
 F 3 "~" V 1150 2950 50  0001 C CNN
 	1    1150 2950
@@
 AR Path="/5E309501/5E62C9E3/5E326A2E" Ref="D57"  Part="1"
 AR Path="/5E309501/5E6352C9/5E326A2E" Ref="D77"  Part="1"
-F 0 "D17" H 1700 3045 50  0000 C CNN
+F 0 "D37" H 1700 3045 50  0000 C CNN
 F 1 "LED_Small_ALT" H 1700 3136 50  0000 C CNN
-F 2 "LED_THT:LED_D3.0mm_Clear" V 1700 3250 50  0001 C CNN
+F 2 "LED_THT:LED_D3.0mm_Front" V 1700 3250 50  0001 C CNN
 F 3 "~" V 1700 3250 50  0001 C CNN
 	1    1700 3250
@@
 AR Path="/5E309501/5E62C9E3/5E326A42" Ref="D46"  Part="1"
 AR Path="/5E309501/5E6352C9/5E326A42" Ref="D66"  Part="1"
-F 0 "D6" H 1150 3045 50  0000 C CNN
+F 0 "D26" H 1150 3045 50  0000 C CNN
 F 1 "LED_Small_ALT" H 1150 3136 50  0000 C CNN
-F 2 "LED_THT:LED_D3.0mm_Clear" V 1150 3250 50  0001 C CNN
+F 2 "LED_THT:LED_D3.0mm_Front" V 1150 3250 50  0001 C CNN
 F 3 "~" V 1150 3250 50  0001 C CNN
 	1    1150 3250
@@
 AR Path="/5E309501/5E62C9E3/5E326A50" Ref="D58"  Part="1"
 AR Path="/5E309501/5E6352C9/5E326A50" Ref="D78"  Part="1"
-F 0 "D18" H 1700 3345 50  0000 C CNN
+F 0 "D38" H 1700 3345 50  0000 C CNN
 F 1 "LED_Small_ALT" H 1700 3436 50  0000 C CNN
-F 2 "LED_THT:LED_D3.0mm_Clear" V 1700 3550 50  0001 C CNN
+F 2 "LED_THT:LED_D3.0mm_Front" V 1700 3550 50  0001 C CNN
 F 3 "~" V 1700 3550 50  0001 C CNN
 	1    1700 3550
@@
 AR Path="/5E309501/5E62C9E3/5E32AAD4" Ref="D59"  Part="1"
 AR Path="/5E309501/5E6352C9/5E32AAD4" Ref="D79"  Part="1"
-F 0 "D19" H 1700 3645 50  0000 C CNN
+F 0 "D39" H 1700 3645 50  0000 C CNN
 F 1 "LED_Small_ALT" H 1700 3736 50  0000 C CNN
-F 2 "LED_THT:LED_D3.0mm_Clear" V 1700 3850 50  0001 C CNN
+F 2 "LED_THT:LED_D3.0mm_Front" V 1700 3850 50  0001 C CNN
 F 3 "~" V 1700 3850 50  0001 C CNN
 	1    1700 3850
@@
 AR Path="/5E309501/5E62C9E3/5E32AAE8" Ref="D47"  Part="1"
 AR Path="/5E309501/5E6352C9/5E32AAE8" Ref="D67"  Part="1"
-F 0 "D7" H 1150 3645 50  0000 C CNN
+F 0 "D27" H 1150 3645 50  0000 C CNN
 F 1 "LED_Small_ALT" H 1150 3736 50  0000 C CNN
-F 2 "LED_THT:LED_D3.0mm_Clear" V 1150 3850 50  0001 C CNN
+F 2 "LED_THT:LED_D3.0mm_Front" V 1150 3850 50  0001 C CNN
 F 3 "~" V 1150 3850 50  0001 C CNN
 	1    1150 3850
@@
 AR Path="/5E309501/5E62C9E3/5E32AAF7" Ref="D61"  Part="1"
 AR Path="/5E309501/5E6352C9/5E32AAF7" Ref="D81"  Part="1"
-F 0 "D21" H 1700 4195 50  0000 C CNN
+F 0 "D41" H 1700 4195 50  0000 C CNN
 F 1 "LED_Small_ALT" H 1700 4286 50  0000 C CNN
-F 2 "LED_THT:LED_D3.0mm_Clear" V 1700 4400 50  0001 C CNN
+F 2 "LED_THT:LED_D3.0mm_Front" V 1700 4400 50  0001 C CNN
 F 3 "~" V 1700 4400 50  0001 C CNN
 	1    1700 4400
@@
 AR Path="/5E309501/5E62C9E3/5E32AB0B" Ref="D48"  Part="1"
 AR Path="/5E309501/5E6352C9/5E32AB0B" Ref="D68"  Part="1"
-F 0 "D8" H 1150 4195 50  0000 C CNN
+F 0 "D28" H 1150 4195 50  0000 C CNN
 F 1 "LED_Small_ALT" H 1150 4286 50  0000 C CNN
-F 2 "LED_THT:LED_D3.0mm_Clear" V 1150 4400 50  0001 C CNN
+F 2 "LED_THT:LED_D3.0mm_Front" V 1150 4400 50  0001 C CNN
 F 3 "~" V 1150 4400 50  0001 C CNN
 	1    1150 4400
@@
 AR Path="/5E309501/5E62C9E3/5E32F97B" Ref="D62"  Part="1"
 AR Path="/5E309501/5E6352C9/5E32F97B" Ref="D82"  Part="1"
-F 0 "D22" H 1700 4495 50  0000 C CNN
+F 0 "D42" H 1700 4495 50  0000 C CNN
 F 1 "LED_Small_ALT" H 1700 4586 50  0000 C CNN
-F 2 "LED_THT:LED_D3.0mm_Clear" V 1700 4700 50  0001 C CNN
+F 2 "LED_THT:LED_D3.0mm_Front" V 1700 4700 50  0001 C CNN
 F 3 "~" V 1700 4700 50  0001 C CNN
 	1    1700 4700
@@
 AR Path="/5E309501/5E62C9E3/5E32F98F" Ref="D49"  Part="1"
 AR Path="/5E309501/5E6352C9/5E32F98F" Ref="D69"  Part="1"
-F 0 "D9" H 1150 4495 50  0000 C CNN
+F 0 "D29" H 1150 4495 50  0000 C CNN
 F 1 "LED_Small_ALT" H 1150 4586 50  0000 C CNN
-F 2 "LED_THT:LED_D3.0mm_Clear" V 1150 4700 50  0001 C CNN
+F 2 "LED_THT:LED_D3.0mm_Front" V 1150 4700 50  0001 C CNN
 F 3 "~" V 1150 4700 50  0001 C CNN
 	1    1150 4700
@@
 AR Path="/5E309501/5E62C9E3/5E3413CA" Ref="D60"  Part="1"
 AR Path="/5E309501/5E6352C9/5E3413CA" Ref="D80"  Part="1"
-F 0 "D20" H 1700 3945 50  0000 C CNN
+F 0 "D40" H 1700 3945 50  0000 C CNN
 F 1 "LED_Small_ALT" H 1700 4036 50  0000 C CNN
-F 2 "LED_THT:LED_D3.0mm_Clear" V 1700 4150 50  0001 C CNN
+F 2 "LED_THT:LED_D3.0mm_Front" V 1700 4150 50  0001 C CNN
 F 3 "~" V 1700 4150 50  0001 C CNN
 	1    1700 4150
@@
 AR Path="/5E309501/5E62C9E3/5E3917E4" Ref="D52"  Part="1"
 AR Path="/5E309501/5E6352C9/5E3917E4" Ref="D72"  Part="1"
-F 0 "D12" H 1700 1445 50  0000 C CNN
+F 0 "D32" H 1700 1445 50  0000 C CNN
 F 1 "LED_Small_ALT" H 1700 1536 50  0000 C CNN
-F 2 "LED_THT:LED_D3.0mm_Clear" V 1700 1650 50  0001 C CNN
+F 2 "LED_THT:LED_D3.0mm_Front" V 1700 1650 50  0001 C CNN
 F 3 "~" V 1700 1650 50  0001 C CNN
 	1    1700 1650

Commit message: joo
Changed lines of the file:
@@
 $Descr A4 11693 8268
 encoding utf-8
-Sheet 18 22
+Sheet 19 22
 Title ""
 Date ""
@@
 AR Path="/5E309501/5E62C9E3/5E30964F" Ref="D50"  Part="1"
 AR Path="/5E309501/5E6352C9/5E30964F" Ref="D70"  Part="1"
-F 0 "D30" H 1700 695 50  0000 C CNN
+F 0 "D50" H 1700 695 50  0000 C CNN
 F 1 "LED_Small_ALT" H 1700 786 50  0000 C CNN
 F 2 "LED_THT:LED_D3.0mm_Front" V 1700 900 50  0001 C CNN
@@
 AR Path="/5E309501/5E62C9E3/5E3126CB" Ref="D51"  Part="1"
 AR Path="/5E309501/5E6352C9/5E3126CB" Ref="D71"  Part="1"
-F 0 "D31" H 1700 1045 50  0000 C CNN
+F 0 "D51" H 1700 1045 50  0000 C CNN
 F 1 "LED_Small_ALT" H 1700 1136 50  0000 C CNN
 F 2 "LED_THT:LED_D3.0mm_Front" V 1700 1250 50  0001 C CNN
@@
 AR Path="/5E309501/5E62C9E3/5E3131D5" Ref="D53"  Part="1"
 AR Path="/5E309501/5E6352C9/5E3131D5" Ref="D73"  Part="1"
-F 0 "D33" H 1700 1845 50  0000 C CNN
+F 0 "D53" H 1700 1845 50  0000 C CNN
 F 1 "LED_Small_ALT" H 1700 1936 50  0000 C CNN
 F 2 "LED_THT:LED_D3.0mm_Front" V 1700 2050 50  0001 C CNN
@@
 AR Path="/5E309501/5E62C9E3/5E314557" Ref="D43"  Part="1"
 AR Path="/5E309501/5E6352C9/5E314557" Ref="D63"  Part="1"
-F 0 "D23" H 1150 1845 50  0000 C CNN
+F 0 "D43" H 1150 1845 50  0000 C CNN
 F 1 "LED_Small_ALT" H 1150 1936 50  0000 C CNN
 F 2 "LED_THT:LED_D3.0mm_Front" V 1150 2050 50  0001 C CNN
@@
 AR Path="/5E309501/5E62C9E3/5E31CE52" Ref="D54"  Part="1"
 AR Path="/5E309501/5E6352C9/5E31CE52" Ref="D74"  Part="1"
-F 0 "D34" H 1700 2145 50  0000 C CNN
+F 0 "D54" H 1700 2145 50  0000 C CNN
 F 1 "LED_Small_ALT" H 1700 2236 50  0000 C CNN
 F 2 "LED_THT:LED_D3.0mm_Front" V 1700 2350 50  0001 C CNN
@@
 AR Path="/5E309501/5E62C9E3/5E31F6AD" Ref="D55"  Part="1"
 AR Path="/5E309501/5E6352C9/5E31F6AD" Ref="D75"  Part="1"
-F 0 "D35" H 1700 2445 50  0000 C CNN
+F 0 "D55" H 1700 2445 50  0000 C CNN
 F 1 "LED_Small_ALT" H 1700 2536 50  0000 C CNN
 F 2 "LED_THT:LED_D3.0mm_Front" V 1700 2650 50  0001 C CNN
@@
 AR Path="/5E309501/5E62C9E3/5E31F6C1" Ref="D44"  Part="1"
 AR Path="/5E309501/5E6352C9/5E31F6C1" Ref="D64"  Part="1"
-F 0 "D24" H 1150 2445 50  0000 C CNN
+F 0 "D44" H 1150 2445 50  0000 C CNN
 F 1 "LED_Small_ALT" H 1150 2536 50  0000 C CNN
 F 2 "LED_THT:LED_D3.0mm_Front" V 1150 2650 50  0001 C CNN
@@
 AR Path="/5E309501/5E62C9E3/5E323EBF" Ref="D56"  Part="1"
 AR Path="/5E309501/5E6352C9/5E323EBF" Ref="D76"  Part="1"
-F 0 "D36" H 1700 2745 50  0000 C CNN
+F 0 "D56" H 1700 2745 50  0000 C CNN
 F 1 "LED_Small_ALT" H 1700 2836 50  0000 C CNN
 F 2 "LED_THT:LED_D3.0mm_Front" V 1700 2950 50  0001 C CNN
@@
 AR Path="/5E309501/5E62C9E3/5E323ED3" Ref="D45"  Part="1"
 AR Path="/5E309501/5E6352C9/5E323ED3" Ref="D65"  Part="1"
-F 0 "D25" H 1150 2745 50  0000 C CNN
+F 0 "D45" H 1150 2745 50  0000 C CNN
 F 1 "LED_Small_ALT" H 1150 2836 50  0000 C CNN
 F 2 "LED_THT:LED_D3.0mm_Front" V 1150 2950 50  0001 C CNN
@@
 AR Path="/5E309501/5E62C9E3/5E326A2E" Ref="D57"  Part="1"
 AR Path="/5E309501/5E6352C9/5E326A2E" Ref="D77"  Part="1"
-F 0 "D37" H 1700 3045 50  0000 C CNN
+F 0 "D57" H 1700 3045 50  0000 C CNN
 F 1 "LED_Small_ALT" H 1700 3136 50  0000 C CNN
 F 2 "LED_THT:LED_D3.0mm_Front" V 1700 3250 50  0001 C CNN
@@
 AR Path="/5E309501/5E62C9E3/5E326A42" Ref="D46"  Part="1"
 AR Path="/5E309501/5E6352C9/5E326A42" Ref="D66"  Part="1"
-F 0 "D26" H 1150 3045 50  0000 C CNN
+F 0 "D46" H 1150 3045 50  0000 C CNN
 F 1 "LED_Small_ALT" H 1150 3136 50  0000 C CNN
 F 2 "LED_THT:LED_D3.0mm_Front" V 1150 3250 50  0001 C CNN
@@
 AR Path="/5E309501/5E62C9E3/5E326A50" Ref="D58"  Part="1"
 AR Path="/5E309501/5E6352C9/5E326A50" Ref="D78"  Part="1"
-F 0 "D38" H 1700 3345 50  0000 C CNN
+F 0 "D58" H 1700 3345 50  0000 C CNN
 F 1 "LED_Small_ALT" H 1700 3436 50  0000 C CNN
 F 2 "LED_THT:LED_D3.0mm_Front" V 1700 3550 50  0001 C CNN
@@
 AR Path="/5E309501/5E62C9E3/5E32AAD4" Ref="D59"  Part="1"
 AR Path="/5E309501/5E6352C9/5E32AAD4" Ref="D79"  Part="1"
-F 0 "D39" H 1700 3645 50  0000 C CNN
+F 0 "D59" H 1700 3645 50  0000 C CNN
 F 1 "LED_Small_ALT" H 1700 3736 50  0000 C CNN
 F 2 "LED_THT:LED_D3.0mm_Front" V 1700 3850 50  0001 C CNN
@@
 AR Path="/5E309501/5E62C9E3/5E32AAE8" Ref="D47"  Part="1"
 AR Path="/5E309501/5E6352C9/5E32AAE8" Ref="D67"  Part="1"
-F 0 "D27" H 1150 3645 50  0000 C CNN
+F 0 "D47" H 1150 3645 50  0000 C CNN
 F 1 "LED_Small_ALT" H 1150 3736 50  0000 C CNN
 F 2 "LED_THT:LED_D3.0mm_Front" V 1150 3850 50  0001 C CNN
@@
 AR Path="/5E309501/5E62C9E3/5E32AAF7" Ref="D61"  Part="1"
 AR Path="/5E309501/5E6352C9/5E32AAF7" Ref="D81"  Part="1"
-F 0 "D41" H 1700 4195 50  0000 C CNN
+F 0 "D61" H 1700 4195 50  0000 C CNN
 F 1 "LED_Small_ALT" H 1700 4286 50  0000 C CNN
 F 2 "LED_THT:LED_D3.0mm_Front" V 1700 4400 50  0001 C CNN
@@
 AR Path="/5E309501/5E62C9E3/5E32AB0B" Ref="D48"  Part="1"
 AR Path="/5E309501/5E6352C9/5E32AB0B" Ref="D68"  Part="1"
-F 0 "D28" H 1150 4195 50  0000 C CNN
+F 0 "D48" H 1150 4195 50  0000 C CNN
 F 1 "LED_Small_ALT" H 1150 4286 50  0000 C CNN
 F 2 "LED_THT:LED_D3.0mm_Front" V 1150 4400 50  0001 C CNN
@@
 AR Path="/5E309501/5E62C9E3/5E32F97B" Ref="D62"  Part="1"
 AR Path="/5E309501/5E6352C9/5E32F97B" Ref="D82"  Part="1"
-F 0 "D42" H 1700 4495 50  0000 C CNN
+F 0 "D62" H 1700 4495 50  0000 C CNN
 F 1 "LED_Small_ALT" H 1700 4586 50  0000 C CNN
 F 2 "LED_THT:LED_D3.0mm_Front" V 1700 4700 50  0001 C CNN
@@
 AR Path="/5E309501/5E62C9E3/5E32F98F" Ref="D49"  Part="1"
 AR Path="/5E309501/5E6352C9/5E32F98F" Ref="D69"  Part="1"
-F 0 "D29" H 1150 4495 50  0000 C CNN
+F 0 "D49" H 1150 4495 50  0000 C CNN
 F 1 "LED_Small_ALT" H 1150 4586 50  0000 C CNN
 F 2 "LED_THT:LED_D3.0mm_Front" V 1150 4700 50  0001 C CNN
@@
 AR Path="/5E309501/5E62C9E3/5E3413CA" Ref="D60"  Part="1"
 AR Path="/5E309501/5E6352C9/5E3413CA" Ref="D80"  Part="1"
-F 0 "D40" H 1700 3945 50  0000 C CNN
+F 0 "D60" H 1700 3945 50  0000 C CNN
 F 1 "LED_Small_ALT" H 1700 4036 50  0000 C CNN
 F 2 "LED_THT:LED_D3.0mm_Front" V 1700 4150 50  0001 C CNN
@@
 AR Path="/5E309501/5E62C9E3/5E3917E4" Ref="D52"  Part="1"
 AR Path="/5E309501/5E6352C9/5E3917E4" Ref="D72"  Part="1"
-F 0 "D32" H 1700 1445 50  0000 C CNN
+F 0 "D52" H 1700 1445 50  0000 C CNN
 F 1 "LED_Small_ALT" H 1700 1536 50  0000 C CNN
 F 2 "LED_THT:LED_D3.0mm_Front" V 1700 1650 50  0001 C CNN

Commit message: joo
Changed lines of the file:
@@
 AR Path="/5E309501/5E62C9E3/5E30964F" Ref="D50"  Part="1"
 AR Path="/5E309501/5E6352C9/5E30964F" Ref="D70"  Part="1"
-F 0 "D50" H 1700 695 50  0000 C CNN
+F 0 "D70" H 1700 695 50  0000 C CNN
 F 1 "LED_Small_ALT" H 1700 786 50  0000 C CNN
 F 2 "LED_THT:LED_D3.0mm_Front" V 1700 900 50  0001 C CNN
@@
 AR Path="/5E309501/5E62C9E3/5E3126CB" Ref="D51"  Part="1"
 AR Path="/5E309501/5E6352C9/5E3126CB" Ref="D71"  Part="1"
-F 0 "D51" H 1700 1045 50  0000 C CNN
+F 0 "D71" H 1700 1045 50  0000 C CNN
 F 1 "LED_Small_ALT" H 1700 1136 50  0000 C CNN
 F 2 "LED_THT:LED_D3.0mm_Front" V 1700 1250 50  0001 C CNN
@@
 AR Path="/5E309501/5E62C9E3/5E3131D5" Ref="D53"  Part="1"
 AR Path="/5E309501/5E6352C9/5E3131D5" Ref="D73"  Part="1"
-F 0 "D53" H 1700 1845 50  0000 C CNN
+F 0 "D73" H 1700 1845 50  0000 C CNN
 F 1 "LED_Small_ALT" H 1700 1936 50  0000 C CNN
 F 2 "LED_THT:LED_D3.0mm_Front" V 1700 2050 50  0001 C CNN
@@
 AR Path="/5E309501/5E62C9E3/5E314557" Ref="D43"  Part="1"
 AR Path="/5E309501/5E6352C9/5E314557" Ref="D63"  Part="1"
-F 0 "D43" H 1150 1845 50  0000 C CNN
+F 0 "D63" H 1150 1845 50  0000 C CNN
 F 1 "LED_Small_ALT" H 1150 1936 50  0000 C CNN
 F 2 "LED_THT:LED_D3.0mm_Front" V 1150 2050 50  0001 C CNN
@@
 AR Path="/5E309501/5E62C9E3/5E31CE52" Ref="D54"  Part="1"
 AR Path="/5E309501/5E6352C9/5E31CE52" Ref="D74"  Part="1"
-F 0 "D54" H 1700 2145 50  0000 C CNN
+F 0 "D74" H 1700 2145 50  0000 C CNN
 F 1 "LED_Small_ALT" H 1700 2236 50  0000 C CNN
 F 2 "LED_THT:LED_D3.0mm_Front" V 1700 2350 50  0001 C CNN
@@
 AR Path="/5E309501/5E62C9E3/5E31F6AD" Ref="D55"  Part="1"
 AR Path="/5E309501/5E6352C9/5E31F6AD" Ref="D75"  Part="1"
-F 0 "D55" H 1700 2445 50  0000 C CNN
+F 0 "D75" H 1700 2445 50  0000 C CNN
 F 1 "LED_Small_ALT" H 1700 2536 50  0000 C CNN
 F 2 "LED_THT:LED_D3.0mm_Front" V 1700 2650 50  0001 C CNN
@@
 AR Path="/5E309501/5E62C9E3/5E31F6C1" Ref="D44"  Part="1"
 AR Path="/5E309501/5E6352C9/5E31F6C1" Ref="D64"  Part="1"
-F 0 "D44" H 1150 2445 50  0000 C CNN
+F 0 "D64" H 1150 2445 50  0000 C CNN
 F 1 "LED_Small_ALT" H 1150 2536 50  0000 C CNN
 F 2 "LED_THT:LED_D3.0mm_Front" V 1150 2650 50  0001 C CNN
@@
 AR Path="/5E309501/5E62C9E3/5E323EBF" Ref="D56"  Part="1"
 AR Path="/5E309501/5E6352C9/5E323EBF" Ref="D76"  Part="1"
-F 0 "D56" H 1700 2745 50  0000 C CNN
+F 0 "D76" H 1700 2745 50  0000 C CNN
 F 1 "LED_Small_ALT" H 1700 2836 50  0000 C CNN
 F 2 "LED_THT:LED_D3.0mm_Front" V 1700 2950 50  0001 C CNN
@@
 AR Path="/5E309501/5E62C9E3/5E323ED3" Ref="D45"  Part="1"
 AR Path="/5E309501/5E6352C9/5E323ED3" Ref="D65"  Part="1"
-F 0 "D45" H 1150 2745 50  0000 C CNN
+F 0 "D65" H 1150 2745 50  0000 C CNN
 F 1 "LED_Small_ALT" H 1150 2836 50  0000 C CNN
 F 2 "LED_THT:LED_D3.0mm_Front" V 1150 2950 50  0001 C CNN
@@
 AR Path="/5E309501/5E62C9E3/5E326A2E" Ref="D57"  Part="1"
 AR Path="/5E309501/5E6352C9/5E326A2E" Ref="D77"  Part="1"
-F 0 "D57" H 1700 3045 50  0000 C CNN
+F 0 "D77" H 1700 3045 50  0000 C CNN
 F 1 "LED_Small_ALT" H 1700 3136 50  0000 C CNN
 F 2 "LED_THT:LED_D3.0mm_Front" V 1700 3250 50  0001 C CNN
@@
 AR Path="/5E309501/5E62C9E3/5E326A42" Ref="D46"  Part="1"
 AR Path="/5E309501/5E6352C9/5E326A42" Ref="D66"  Part="1"
-F 0 "D46" H 1150 3045 50  0000 C CNN
+F 0 "D66" H 1150 3045 50  0000 C CNN
 F 1 "LED_Small_ALT" H 1150 3136 50  0000 C CNN
 F 2 "LED_THT:LED_D3.0mm_Front" V 1150 3250 50  0001 C CNN
@@
 AR Path="/5E309501/5E62C9E3/5E326A50" Ref="D58"  Part="1"
 AR Path="/5E309501/5E6352C9/5E326A50" Ref="D78"  Part="1"
-F 0 "D58" H 1700 3345 50  0000 C CNN
+F 0 "D78" H 1700 3345 50  0000 C CNN
 F 1 "LED_Small_ALT" H 1700 3436 50  0000 C CNN
 F 2 "LED_THT:LED_D3.0mm_Front" V 1700 3550 50  0001 C CNN
@@
 AR Path="/5E309501/5E62C9E3/5E32AAD4" Ref="D59"  Part="1"
 AR Path="/5E309501/5E6352C9/5E32AAD4" Ref="D79"  Part="1"
-F 0 "D59" H 1700 3645 50  0000 C CNN
+F 0 "D79" H 1700 3645 50  0000 C CNN
 F 1 "LED_Small_ALT" H 1700 3736 50  0000 C CNN
 F 2 "LED_THT:LED_D3.0mm_Front" V 1700 3850 50  0001 C CNN
@@
 AR Path="/5E309501/5E62C9E3/5E32AAE8" Ref="D47"  Part="1"
 AR Path="/5E309501/5E6352C9/5E32AAE8" Ref="D67"  Part="1"
-F 0 "D47" H 1150 3645 50  0000 C CNN
+F 0 "D67" H 1150 3645 50  0000 C CNN
 F 1 "LED_Small_ALT" H 1150 3736 50  0000 C CNN
 F 2 "LED_THT:LED_D3.0mm_Front" V 1150 3850 50  0001 C CNN
@@
 AR Path="/5E309501/5E62C9E3/5E32AAF7" Ref="D61"  Part="1"
 AR Path="/5E309501/5E6352C9/5E32AAF7" Ref="D81"  Part="1"
-F 0 "D61" H 1700 4195 50  0000 C CNN
+F 0 "D81" H 1700 4195 50  0000 C CNN
 F 1 "LED_Small_ALT" H 1700 4286 50  0000 C CNN
 F 2 "LED_THT:LED_D3.0mm_Front" V 1700 4400 50  0001 C CNN
@@
 AR Path="/5E309501/5E62C9E3/5E32AB0B" Ref="D48"  Part="1"
 AR Path="/5E309501/5E6352C9/5E32AB0B" Ref="D68"  Part="1"
-F 0 "D48" H 1150 4195 50  0000 C CNN
+F 0 "D68" H 1150 4195 50  0000 C CNN
 F 1 "LED_Small_ALT" H 1150 4286 50  0000 C CNN
 F 2 "LED_THT:LED_D3.0mm_Front" V 1150 4400 50  0001 C CNN
@@
 AR Path="/5E309501/5E62C9E3/5E32F97B" Ref="D62"  Part="1"
 AR Path="/5E309501/5E6352C9/5E32F97B" Ref="D82"  Part="1"
-F 0 "D62" H 1700 4495 50  0000 C CNN
+F 0 "D82" H 1700 4495 50  0000 C CNN
 F 1 "LED_Small_ALT" H 1700 4586 50  0000 C CNN
 F 2 "LED_THT:LED_D3.0mm_Front" V 1700 4700 50  0001 C CNN
@@
 AR Path="/5E309501/5E62C9E3/5E32F98F" Ref="D49"  Part="1"
 AR Path="/5E309501/5E6352C9/5E32F98F" Ref="D69"  Part="1"
-F 0 "D49" H 1150 4495 50  0000 C CNN
+F 0 "D69" H 1150 4495 50  0000 C CNN
 F 1 "LED_Small_ALT" H 1150 4586 50  0000 C CNN
 F 2 "LED_THT:LED_D3.0mm_Front" V 1150 4700 50  0001 C CNN
@@
 AR Path="/5E309501/5E62C9E3/5E3413CA" Ref="D60"  Part="1"
 AR Path="/5E309501/5E6352C9/5E3413CA" Ref="D80"  Part="1"
-F 0 "D60" H 1700 3945 50  0000 C CNN
+F 0 "D80" H 1700 3945 50  0000 C CNN
 F 1 "LED_Small_ALT" H 1700 4036 50  0000 C CNN
 F 2 "LED_THT:LED_D3.0mm_Front" V 1700 4150 50  0001 C CNN
@@
 AR Path="/5E309501/5E62C9E3/5E3917E4" Ref="D52"  Part="1"
 AR Path="/5E309501/5E6352C9/5E3917E4" Ref="D72"  Part="1"
-F 0 "D52" H 1700 1445 50  0000 C CNN
+F 0 "D72" H 1700 1445 50  0000 C CNN
 F 1 "LED_Small_ALT" H 1700 1536 50  0000 C CNN
 F 2 "LED_THT:LED_D3.0mm_Front" V 1700 1650 50  0001 C CNN
