File: kello-zcdetector/_autosave-kello-zcdetector.sch (KiCad schematic (older format))
At the start: 9 parts, among them J1 Conn_01x02_Male, J2 Conn_01x02_Male, U1 LTV-817S

Commit message: joo
Parts:
- added F2: Fuse, Fuse:Fuse_10mmx3mm, symbol Device:Fuse
- gave numbers to parts that had none: 1
Connections:
- net at R1.2: now also F2.2; no longer J1.1 (Pin_1)
- new net: F2.1, J1.1 (Pin_1)
Changed lines of the file:
@@
 $EndComp
-Wire Wire Line
-	1650 3150 1950 3150
 Wire Wire Line
 	1650 3250 1800 3250
@@
 	5050 3200 5200 3200
 $Comp
-L Device:Fuse F?
+L Device:Fuse F1
 U 1 1 5E4EBF45
 P 1800 3400
-F 0 "F?" H 1740 3354 50  0000 R CNN
+F 0 "F1" H 1740 3354 50  0000 R CNN
 F 1 "Fuse" H 1740 3445 50  0000 R CNN
 F 2 "Fuse:Fuse_10mmx3mm" V 1730 3400 50  0001 C CNN
@@
 Wire Wire Line
 	1800 3550 1950 3550
+$Comp
+L Device:Fuse F2
+U 1 1 5EDDD343
+P 1800 3150
+F 0 "F2" H 1740 3104 50  0000 R CNN
+F 1 "Fuse" H 1740 3195 50  0000 R CNN
+F 2 "Fuse:Fuse_10mmx3mm" V 1730 3150 50  0001 C CNN
+F 3 "~" H 1800 3150 50  0001 C CNN
+	1    1800 3150
+	0    -1   -1   0
+$EndComp
 $EndSCHEMATC
