File: kello-zcdetector/kello-zcdetector.kicad_pcb (KiCad board)
At the start: 2 copper layers, 8 parts, among them J1 Conn_01x02_Male, J2 Conn_01x02_Male, U1 LTV-817S

Commit message: joo
Parts:
- R1, R2, R3, R4: footprint Resistor_SMD:R_1206_3216Metric -> Resistor_SMD:R_0805_2012Metric

Commit message: joo
Parts:
- added F1: Fuse, Fuse:Fuse_10mmx3mm, F.Cu at (17.6, 14.4)
- added F2: Fuse, Fuse:Fuse_10mmx3mm, F.Cu at (17.6, 25.0)
- moved U1 9.72 mm to (39.8, 23.7)
- moved R3 9.15 mm to (32.6, 13.6), turned to 90 degrees
- moved R1 8.64 mm to (19.7, 22.0), turned to 0 degrees
- moved J2 7.88 mm to (44.8, 16.4), turned to 0 degrees
- moved R4 7.47 mm to (27.8, 13.6), turned to 90 degrees
- moved J1 6.98 mm to (14.0, 21.0), turned to 180 degrees
- moved D1 4.17 mm to (29.1, 21.0), turned to 90 degrees
- moved R2 1.45 mm to (19.7, 17.4), turned to 0 degrees
Connections:
- J1 pad 1: Net-(J1-Pad1) -> Net-(F2-Pad1)
- J1 pad 2: Net-(J1-Pad2) -> Net-(F1-Pad2)
- R1 pad 2: Net-(J1-Pad1) -> Net-(F2-Pad2)
- R2 pad 2: Net-(J1-Pad2) -> Net-(F1-Pad1)
Routing:
- net Net-(R1-Pad1): track 2.33 -> 20.3 mm
- net Net-(R2-Pad1): track 4.13 -> 14.1 mm
- net Net-(J2-Pad1): track 3.49 -> 9.94 mm
- net Net-(F2-Pad1): track 0.00 -> 4.14 mm
- net Net-(F1-Pad2): track 0.00 -> 4.14 mm
- net Net-(F2-Pad2): track 0.00 -> 3.70 mm
- net Net-(F1-Pad1): track 0.00 -> 3.70 mm
- net Net-(J1-Pad1): track 3.26 -> 0.00 mm
- net Net-(J1-Pad2): track 3.12 -> 0.00 mm
- net Net-(D1-Pad1): track 13.6 -> 10.5 mm
- net Net-(D1-Pad3): track 4.17 -> 2.48 mm
- net Net-(D1-Pad4): track 3.65 -> 2.59 mm

Commit message: diodisillalla zcdet
Parts:
- moved R2 6.83 mm to (24.8, 12.8), turned to 180 degrees
Routing:
- net Net-(R2-Pad1): track 14.1 -> 2.18 mm
- net Net-(F1-Pad1): track 3.70 -> 2.87 mm
Changed lines of the file:
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@@
     (thickness 1.6)
     (drawings 0)
-    (tracks 40)
+    (tracks 34)
     (zones 0)
     (modules 10)
@@
   )
   (module Resistor_SMD:R_0805_2012Metric (layer F.Cu)
-    (at 19.685 17.399)
+    (at 24.765 12.827 180)
     (descr "Resistor SMD 0805 (2012 Metric), square (rectangular) end terminal, IPC_7351 nominal, (Body size source: https://docs.google.com/spreadsheets/d/1BsfQQcO9C6DZCsRaXUlFlo91Tg2WpOkGARC1WS5S8t0/edit?usp=sharing), generated with kicad-footprint-generator")
     (tags resistor)
@@
     (fp_line (start -1 -0.6) (end 1 -0.6) (layer F.Fab) (width 0.1))
     (fp_line (start -1 0.6) (end -1 -0.6) (layer F.Fab) (width 0.1))
-    (pad 2 smd roundrect (at 0.9375 0) (size 0.975 1.4) (layers F.Cu F.Paste F.Mask) (roundrect_rratio 0.25)
+    (pad 2 smd roundrect (at 0.9375 0 180) (size 0.975 1.4) (layers F.Cu F.Paste F.Mask) (roundrect_rratio 0.25)
       (net 10 "Net-(F1-Pad1)"))
-    (pad 1 smd roundrect (at -0.9375 0) (size 0.975 1.4) (layers F.Cu F.Paste F.Mask) (roundrect_rratio 0.25)
+    (pad 1 smd roundrect (at -0.9375 0 180) (size 0.975 1.4) (layers F.Cu F.Paste F.Mask) (roundrect_rratio 0.25)
       (net 8 "Net-(R2-Pad1)"))
     (model ${KISYS3DMOD}/Resistor_SMD.3dshapes/R_0805_2012Metric.wrl
@@
   (segment (start 18.7475 21.717) (end 18.7475 21.017) (width 0.5) (layer F.Cu) (net 7))
   (segment (start 27.051 20.447) (end 29.591 17.907) (width 0.5) (layer F.Cu) (net 7))
-  (segment (start 25.9565 12.6515) (end 27.813 12.6515) (width 0.5) (layer F.Cu) (net 8))
-  (segment (start 18.7475 18.353) (end 19.5715 19.177) (width 0.5) (layer F.Cu) (net 8))
-  (segment (start 18.7475 17.653) (end 18.7475 18.353) (width 0.5) (layer F.Cu) (net 8))
-  (segment (start 19.5715 19.177) (end 21.717 19.177) (width 0.5) (layer F.Cu) (net 8))
-  (segment (start 21.717 19.177) (end 23.749 17.145) (width 0.5) (layer F.Cu) (net 8))
-  (segment (start 24.511 14.097) (end 25.9565 12.6515) (width 0.5) (layer F.Cu) (net 8))
-  (segment (start 23.749 17.145) (end 24.511 16.383) (width 0.5) (layer F.Cu) (net 8))
-  (segment (start 24.511 16.383) (end 24.511 14.097) (width 0.5) (layer F.Cu) (net 8))
+  (segment (start 27.6375 12.827) (end 27.813 12.6515) (width 0.5) (layer F.Cu) (net 8))
+  (segment (start 25.7025 12.827) (end 27.6375 12.827) (width 0.5) (layer F.Cu) (net 8))
   (segment (start 13.97 14.542) (end 14.161 14.351) (width 0.5) (layer F.Cu) (net 9))
   (segment (start 13.97 18.415) (end 13.97 14.542) (width 0.5) (layer F.Cu) (net 9))
-  (segment (start 21.589 16.6865) (end 20.6225 17.653) (width 0.5) (layer F.Cu) (net 10))
-  (segment (start 21.589 14.351) (end 21.589 16.6865) (width 0.5) (layer F.Cu) (net 10))
+  (segment (start 23.113 12.827) (end 21.589 14.351) (width 0.5) (layer F.Cu) (net 10))
+  (segment (start 23.8275 12.827) (end 23.113 12.827) (width 0.5) (layer F.Cu) (net 10))
   (segment (start 21.589 22.6835) (end 21.589 25.019) (width 0.5) (layer F.Cu) (net 11))
   (segment (start 20.6225 21.717) (end 21.589 22.6835) (width 0.5) (layer F.Cu) (net 11))

Commit message: diodisillalla zcdet
Parts:
- moved R1 2.81 mm to (22.5, 21.7), turned to 180 degrees
- moved R4 0.25 mm to (27.6, 13.6)
Routing:
- net Net-(R1-Pad1): track 20.3 -> 15.1 mm
Changed lines of the file:
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@@
     (thickness 1.6)
     (drawings 0)
-    (tracks 34)
+    (tracks 33)
     (zones 0)
     (modules 10)
@@
   )
   (module Resistor_SMD:R_0805_2012Metric (layer F.Cu)
-    (at 27.813 13.589 90)
+    (at 27.559 13.589 90)
     (descr "Resistor SMD 0805 (2012 Metric), square (rectangular) end terminal, IPC_7351 nominal, (Body size source: https://docs.google.com/spreadsheets/d/1BsfQQcO9C6DZCsRaXUlFlo91Tg2WpOkGARC1WS5S8t0/edit?usp=sharing), generated with kicad-footprint-generator")
     (tags resistor)
@@
   )
   (module Resistor_SMD:R_0805_2012Metric (layer F.Cu)
-    (at 19.685 21.971)
+    (at 22.479 21.717 180)
     (descr "Resistor SMD 0805 (2012 Metric), square (rectangular) end terminal, IPC_7351 nominal, (Body size source: https://docs.google.com/spreadsheets/d/1BsfQQcO9C6DZCsRaXUlFlo91Tg2WpOkGARC1WS5S8t0/edit?usp=sharing), generated with kicad-footprint-generator")
     (tags resistor)
@@
     (fp_line (start -1 -0.6) (end 1 -0.6) (layer F.Fab) (width 0.1))
     (fp_line (start -1 0.6) (end -1 -0.6) (layer F.Fab) (width 0.1))
-    (pad 2 smd roundrect (at 0.9375 0) (size 0.975 1.4) (layers F.Cu F.Paste F.Mask) (roundrect_rratio 0.25)
+    (pad 2 smd roundrect (at 0.9375 0 180) (size 0.975 1.4) (layers F.Cu F.Paste F.Mask) (roundrect_rratio 0.25)
       (net 11 "Net-(F2-Pad2)"))
-    (pad 1 smd roundrect (at -0.9375 0) (size 0.975 1.4) (layers F.Cu F.Paste F.Mask) (roundrect_rratio 0.25)
+    (pad 1 smd roundrect (at -0.9375 0 180) (size 0.975 1.4) (layers F.Cu F.Paste F.Mask) (roundrect_rratio 0.25)
       (net 7 "Net-(R1-Pad1)"))
     (model ${KISYS3DMOD}/Resistor_SMD.3dshapes/R_0805_2012Metric.wrl
@@
     )
   )
-  (segment (start 27.813 15.305) (end 26.533 16.585) (width 0.5) (layer F.Cu) (net 1))
-  (segment (start 27.813 14.5265) (end 27.813 15.305) (width 0.5) (layer F.Cu) (net 1))
+  (segment (start 26.533 15.5525) (end 27.559 14.5265) (width 0.5) (layer F.Cu) (net 1))
+  (segment (start 26.533 16.585) (end 26.533 15.5525) (width 0.5) (layer F.Cu) (net 1))
   (segment (start 31.633 15.5325) (end 32.639 14.5265) (width 0.5) (layer F.Cu) (net 2))
   (segment (start 31.633 16.585) (end 31.633 15.5325) (width 0.5) (layer F.Cu) (net 2))
@@
   (segment (start 44.676002 25.019) (end 46.101 23.594002) (width 0.5) (layer F.Cu) (net 6))
   (segment (start 44.516 25.019) (end 44.676002 25.019) (width 0.5) (layer F.Cu) (net 6))
+  (segment (start 29.845 13.843) (end 31.0365 12.6515) (width 0.5) (layer F.Cu) (net 7))
   (segment (start 31.0365 12.6515) (end 32.639 12.6515) (width 0.5) (layer F.Cu) (net 7))
-  (segment (start 18.7475 21.017) (end 19.3175 20.447) (width 0.5) (layer F.Cu) (net 7))
-  (segment (start 29.591 14.097) (end 31.0365 12.6515) (width 0.5) (layer F.Cu) (net 7))
-  (segment (start 19.3175 20.447) (end 27.051 20.447) (width 0.5) (layer F.Cu) (net 7))
-  (segment (start 29.591 17.907) (end 29.591 14.097) (width 0.5) (layer F.Cu) (net 7))
-  (segment (start 18.7475 21.717) (end 18.7475 21.017) (width 0.5) (layer F.Cu) (net 7))
-  (segment (start 27.051 20.447) (end 29.591 17.907) (width 0.5) (layer F.Cu) (net 7))
+  (segment (start 29.845 17.399) (end 29.845 13.843) (width 0.5) (layer F.Cu) (net 7))
+  (segment (start 23.4165 21.717) (end 25.527 21.717) (width 0.5) (layer F.Cu) (net 7))
+  (segment (start 25.527 21.717) (end 29.845 17.399) (width 0.5) (layer F.Cu) (net 7))
   (segment (start 27.6375 12.827) (end 27.813 12.6515) (width 0.5) (layer F.Cu) (net 8))
-  (segment (start 25.7025 12.827) (end 27.6375 12.827) (width 0.5) (layer F.Cu) (net 8))
+  (segment (start 27.3835 12.827) (end 27.559 12.6515) (width 0.5) (layer F.Cu) (net 8))
+  (segment (start 25.7025 12.827) (end 27.3835 12.827) (width 0.5) (layer F.Cu) (net 8))
   (segment (start 13.97 14.542) (end 14.161 14.351) (width 0.5) (layer F.Cu) (net 9))
   (segment (start 13.97 18.415) (end 13.97 14.542) (width 0.5) (layer F.Cu) (net 9))
   (segment (start 23.113 12.827) (end 21.589 14.351) (width 0.5) (layer F.Cu) (net 10))
   (segment (start 23.8275 12.827) (end 23.113 12.827) (width 0.5) (layer F.Cu) (net 10))
-  (segment (start 21.589 22.6835) (end 21.589 25.019) (width 0.5) (layer F.Cu) (net 11))
-  (segment (start 20.6225 21.717) (end 21.589 22.6835) (width 0.5) (layer F.Cu) (net 11))
+  (segment (start 21.5415 24.9715) (end 21.589 25.019) (width 0.5) (layer F.Cu) (net 11))
+  (segment (start 21.5415 21.717) (end 21.5415 24.9715) (width 0.5) (layer F.Cu) (net 11))
   (segment (start 13.97 24.828) (end 14.161 25.019) (width 0.5) (layer F.Cu) (net 12))
   (segment (start 13.97 20.955) (end 13.97 24.828) (width 0.5) (layer F.Cu) (net 12))

Commit message: jawohl
Parts:
- added MOUNT: MountingHole_2.2mm_M2, MountingHole:MountingHole_2.2mm_M2, F.Cu at (35.7, 18.2)
- J1: footprint Connector_PinHeader_2.54mm:PinHeader_1x02_P2.54mm_Vertical -> Connector_PinHeader_2.54mm:AC_connector
- moved J2 10.7 mm to (53.2, 23.0)
- moved U1 10.3 mm to (48.4, 18.2)
- moved R3 9.60 mm to (26.8, 21.2), turned to 180 degrees
- moved D1 6.83 mm to (34.2, 25.5), turned to 180 degrees
- moved F2 6.63 mm to (20.2, 31.1)
- moved J1 6.32 mm to (16.4, 26.8)
- moved R4 4.58 mm to (32.1, 13.3), turned to 180 degrees
- moved R1 3.98 mm to (24.3, 25.3), turned to 270 degrees
- moved R2 3.34 mm to (28.1, 13.3)
- moved F1 2.62 mm to (20.2, 14.6)
Routing:
- net Net-(D1-Pad4): track 2.48 -> 17.4 mm
- net Net-(R1-Pad1): track 15.1 -> 3.79 mm
- net Net-(D1-Pad1): track 10.5 -> 19.3 mm
- net Net-(J2-Pad2): track 3.69 -> 11.0 mm
- net Net-(J2-Pad1): track 9.94 -> 3.58 mm
- net Net-(D1-Pad2): track 3.48 -> 7.71 mm
- net Net-(F2-Pad2): track 3.32 -> 5.20 mm
- net Net-(F2-Pad1): track 4.14 -> 5.91 mm
- net Net-(F1-Pad1): track 2.87 -> 3.46 mm
- net Net-(F1-Pad2): track 4.14 -> 4.65 mm
Other:
- board outline added: 45 x 21.6 mm

Commit message: joo
Parts:
- removed the MOUNT at (35.7, 18.2)
- added MOUNT: MountingHole_2.2mm_M2, MountingHole:MountingHole_2.2mm_M2, F.Cu at (40.5, 45.1)
- added MOUNT: MountingHole_2.2mm_M2, MountingHole:MountingHole_2.2mm_M2, F.Cu at (40.5, 14.6)
- added R5: 47k, Resistor_SMD:R_0805_2012Metric, F.Cu at (47.6, 40.0)
- J2: footprint Connector_PinHeader_2.54mm:PinHeader_1x02_P2.54mm_Vertical -> Connector_PinHeader_2.54mm:PinHeader_1x03_P2.54mm_Vertical
- moved R2 33.0 mm to (22.5, 45.8)
- moved R4 33.0 mm to (26.5, 45.8)
- moved F1 27.7 mm to (16.6, 42.0), turned to 90 degrees
- moved F2 13.4 mm to (16.6, 18.2), turned to 270 degrees
- moved R1 11.6 mm to (22.2, 13.8), turned to 180 degrees
- moved J2 10.5 mm to (47.6, 31.9)
- moved U1 10.0 mm to (42.5, 26.3)
- moved D1 8.42 mm to (33.4, 33.9)
- moved J1 7.62 mm to (16.6, 34.4)
- moved R3 7.41 mm to (26.0, 13.8)
Connections:
- J1 pad 1: Net-(F2-Pad1) -> Net-(F1-Pad2)
- J1 pad 2: Net-(F1-Pad2) -> Net-(F2-Pad2)
- R1 pad 2: Net-(F2-Pad2) -> Net-(F2-Pad1)
Routing:
- net Net-(D1-Pad3): track 2.79 -> 18.4 mm
- net Net-(J2-Pad2): track 11.0 -> 19.2 mm
- net Net-(D1-Pad4): track 17.4 -> 10.0 mm
- net Net-(D1-Pad2): track 7.71 -> 3.80 mm
- net Net-(J2-Pad3): track 0.00 -> 3.44 mm
- net Net-(D1-Pad1): track 19.3 -> 16.6 mm
- net Net-(R1-Pad1): track 3.79 -> 1.93 mm
- net Net-(F1-Pad1): track 3.46 -> 4.98 mm
- net Net-(F2-Pad1): track 5.91 -> 4.78 mm
- net Net-(J2-Pad1): track 3.58 -> 4.45 mm
- net Net-(F2-Pad2): track 5.20 -> 4.64 mm
- net Net-(F1-Pad2): track 4.65 -> 4.14 mm
Other:
- board size 45 x 21.6 mm -> 38.6 x 35.6 mm
