File: isp-molex-adapter/isp-molex-adapter.kicad_pcb (KiCad board)
At the start: 2 copper layers, 13 parts, among them J1 AVR-ISP-6, J2 AVR-ISP-10, J3 AVR-ISP-6, Q1 BC850, Q2 BC850

Commit message: tilasin nää
Other:
- board outline added: 24.1 x 14 mm
